File: CAD/eagle/STARduino/starduino.sch (EAGLE design)
At the start: 81 parts, among them J1 MICRO_SD, Q1 BSD223P, U1 ATSAMD21G18, U10 PCA9685, U11 DRV8846RGER, U2 ACS722LLCTR-10AU, U3 ADXL375BCCZ, U4 MAX31725MTA+, U5 HSCMNNN1.6BAAA3, U6 DS3231MZ+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

Commit message: Removed Hacked Motor PWM Driver/Multiplexer
Removed hacked motor PWM driver/multiplexer
Parts:
- removed Q1: BSD223P, transistor-fet:BSD223P
- removed R19: 10k, rcl:R-US_R0603
- removed U10: PCA9685, SparkFun-DigitalIC:PCA9685
Connections:
- removed net N$19: R19.1, U10.EXTCLK
- net +5V: no longer U10.VDD
- net DIR: no longer U10.CH3
- net GND: no longer R19.2, U10.VSS
- net NENBL: no longer U10.CH1
- net NSLEEP: no longer U10.CH2
- net SCL: no longer U10.SCL
- net SDA: no longer U10.SDA
Other:
- note added: "MOTOR DRIVER"
- moved on the sheet: C26, C27, C28, JP5, R10, R11, R12, R13, R14, R15, R16, R17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

Commit message: Added Multiplexer
Added multiplexer for motor driver and assosciated level-shifting
circuitry.
Parts:
- removed R13, R15: 10k, rcl:R-US_R0603
- added R19: 220k, rcl:R-US_R0603
- added R20, R21: 4.7k, rcl:R-US_R0603
- added U10: TCA9535_RTW_24, MotorDriver:TCA9535_RTW_24
- added U12: MC14504BDTG, MotorDriver:MC14504BDTG
- added U13: PCA9306DCT, MotorDriver:PCA9306DCT
- added U14, U15: MC74VHC1GT125DT, MotorDriver:MC74VHC1GT125DT
Connections:
- removed net PA20: R14.2, U1.PA20/EIC/SCOM5PAD2+, U11.NFAULT
- removed net PA21: SJ6.2, U1.PA21/EIC/SCOM5PAD3+
- removed net PA28: SJ5.2, U1.PA28/EIC
- removed net PB02: SJ3.2, U1.PB02/EIC/AIN10/SCOM5PAD0
- removed net PB03: SJ4.2, U1.PB03/EIC/AIN11/SCOM5PAD1
- removed net PB08: SJ1.2, U1.PB08/EIC/AIN2/SCOM4PAD0/TC4
- removed net PB09: SJ2.2, U1.PB09/EIC/AIN3/SCOM4PAD1//TC4
- new net I0: U10.P16, U11.I0
- new net I1: U10.P17, U11.I1
- new net IMDUR: U12.AIN
- new net IMUDR: SJ1.2
- new net IMUINT1: SJ2.2, U12.BIN
- new net IMUINT2: SJ3.2, U12.CIN
- new net IMUINT3: SJ4.2, U12.DIN
- new net IMUINT4: SJ5.2, U12.EIN
- new net IMUINT5: SJ6.2, U12.FIN
- new net IOEINT: U1.PA21/EIC/SCOM5PAD3+, U14.OUTY
- new net M0: U10.P14, U11.M0
- new net M1: U10.P15, U11.M1
- new net N$19: U10.P00, U12.AOUT
- new net N$23: U10.P01, U12.BOUT
- new net N$28: U10.P02, U12.COUT
- new net N$29: U10.P03, U12.DOUT
- new net N$30: U10.P04, U12.EOUT
- new net N$31: U10.P05, U12.FOUT
- new net N$33: R20.1, U10.SDA, U13.SDA2
- new net N$34: R21.1, U10.SCL, U13.SCL2
- new net N$35: R19.1, U13.EN, U13.VREF2
- new net NFAULT: R14.2, U10.P13, U11.NFAULT
- net +3V3: now also U12.VCC, U13.VREF1, U14.VCC
- net +5V: now also R19.2, R20.2, R21.2, U10.A0, U10.A1, U10.A2, U10.VCC, U12.VDD, U15.VCC; no longer R12.2, R15.1
- net DIR: now also U10.P12
- net GND: now also R11.1, R12.1, U10.EPAD, U10.GND, U12.MODE, U12.VSS, U13.GND, U14.GND, U15.GND; no longer R11.2, R13.1
- net N$22: now also U11.STEP, U15.OUTY; no longer R11.1, U11.I0
- net N$24: now also R11.2, U15.!OE!; no longer R15.2, U11.M0
- net N$25: now also U10.INT, U14.INA; no longer R12.1, U11.I1
- net N$27: now also R12.2, U14.!OE!; no longer R13.2, U11.M1
- net NENBL: now also U10.P11
- net NSLEEP: now also U10.P10
- net SCL: now also U13.SCL1
- net SDA: now also U13.SDA1
- net STEPFREQ: now also U1.PB08/EIC/AIN2/SCOM4PAD0/TC4, U15.INA; no longer U11.STEP
Other:
- note added: "MULTIPLEXER"
- moved on the sheet: JP5, R11, R12

Commit message: Renumbered Resistors
Renumbered resistors in motor driver and multiplexer blocks to maintain
consecutive numbering.
Parts:
- removed R20, R21: 4.7k, rcl:R-US_R0603
- added R13, R15: 10k, rcl:R-US_R0603
- R16, R17: value 10k -> 4.7k
- R18: value 10k -> 220k
- R19: value 220k -> 10k
Connections:
- net +5V: now also R12.1, R13.2, R14.2, R15.2; no longer R14.1, R19.2, R20.2, R21.2
- net GND: now also R19.1; no longer R12.1
- net N$16: now also R13.1; no longer R16.1
- net N$17: now also R14.1; no longer R17.1
- net N$18: now also R15.1; no longer R18.1
- net N$27: now also R19.2; no longer R12.2
- net N$33: now also R17.1; no longer R20.1
- net N$34: now also R16.1; no longer R21.1
- net N$35: now also R18.1; no longer R19.1
- net NFAULT: now also R12.2; no longer R14.2
Other:
- moved on the sheet: R12, R14, R16, R17, R18, R19
Changed lines of the file:
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@@
 <part name="P+4" library="supply1" deviceset="+5V" device=""/>
 <part name="C28" library="rcl" deviceset="C-US" device="C0603" value="2.2uF"/>
+<part name="R12" library="rcl" deviceset="R-US_" device="R0603" value="10k"/>
+<part name="P+5" library="supply1" deviceset="+5V" device=""/>
+<part name="R13" library="rcl" deviceset="R-US_" device="R0603" value="10k"/>
 <part name="R14" library="rcl" deviceset="R-US_" device="R0603" value="10k"/>
-<part name="P+5" library="supply1" deviceset="+5V" device=""/>
-<part name="R16" library="rcl" deviceset="R-US_" device="R0603" value="10k"/>
-<part name="R17" library="rcl" deviceset="R-US_" device="R0603" value="10k"/>
-<part name="R18" library="rcl" deviceset="R-US_" device="R0603" value="10k"/>
+<part name="R15" library="rcl" deviceset="R-US_" device="R0603" value="10k"/>
 <part name="U10" library="MotorDriver" deviceset="TCA9535_RTW_24" device=""/>
 <part name="P+6" library="supply1" deviceset="+5V" device=""/>
@@
 <part name="U12" library="MotorDriver" deviceset="MC14504BDTG" device=""/>
 <part name="GND35" library="supply1" deviceset="GND" device=""/>
-<part name="R19" library="rcl" deviceset="R-US_" device="R0603" value="220k"/>
-<part name="R20" library="rcl" deviceset="R-US_" device="R0603" value="4.7k"/>
-<part name="R21" library="rcl" deviceset="R-US_" device="R0603" value="4.7k"/>
+<part name="R18" library="rcl" deviceset="R-US_" device="R0603" value="220k"/>
+<part name="R17" library="rcl" deviceset="R-US_" device="R0603" value="4.7k"/>
+<part name="R16" library="rcl" deviceset="R-US_" device="R0603" value="4.7k"/>
 <part name="+3V16" library="supply1" deviceset="+3V3" device=""/>
 <part name="U13" library="MotorDriver" deviceset="PCA9306" device="DCT"/>
@@
 <part name="U15" library="MotorDriver" deviceset="MC74VHC1GT125" device="DT"/>
 <part name="R11" library="rcl" deviceset="R-US_" device="R0603" value="10k"/>
-<part name="R12" library="rcl" deviceset="R-US_" device="R0603" value="10k"/>
+<part name="R19" library="rcl" deviceset="R-US_" device="R0603" value="10k"/>
 <part name="+3V17" library="supply1" deviceset="+3V3" device=""/>
 </parts>
@@
 </instance>
 <instance part="C28" gate="G$1" x="335.28" y="-86.36"/>
-<instance part="R14" gate="G$1" x="264.16" y="-88.9"/>
+<instance part="R12" gate="G$1" x="264.16" y="-88.9"/>
 <instance part="P+5" gate="1" x="259.08" y="-81.28" smashed="yes">
 <attribute name="VALUE" x="266.7" y="-81.28" size="1.778" layer="96" rot="R180"/>
 </instance>
-<instance part="R16" gate="G$1" x="353.06" y="-101.6"/>
-<instance part="R17" gate="G$1" x="342.9" y="-109.22"/>
-<instance part="R18" gate="G$1" x="350.52" y="-114.3"/>
+<instance part="R13" gate="G$1" x="353.06" y="-101.6"/>
+<instance part="R14" gate="G$1" x="342.9" y="-109.22"/>
+<instance part="R15" gate="G$1" x="350.52" y="-114.3"/>
 <instance part="U10" gate="A" x="269.24" y="-147.32"/>
 <instance part="P+6" gate="1" x="330.2" y="-142.24" smashed="yes">
@@
 <instance part="U12" gate="G$1" x="243.84" y="-160.02"/>
 <instance part="GND35" gate="1" x="391.16" y="-152.4"/>
-<instance part="R19" gate="G$1" x="337.82" y="-152.4" rot="R180"/>
-<instance part="R20" gate="G$1" x="342.9" y="-170.18" rot="R270"/>
-<instance part="R21" gate="G$1" x="335.28" y="-170.18" rot="R270"/>
+<instance part="R18" gate="G$1" x="337.82" y="-152.4" rot="R180"/>
+<instance part="R17" gate="G$1" x="342.9" y="-170.18" rot="R270"/>
+<instance part="R16" gate="G$1" x="335.28" y="-170.18" rot="R270"/>
 <instance part="+3V16" gate="G$1" x="388.62" y="-154.94" smashed="yes">
 <attribute name="VALUE" x="386.08" y="-154.94" size="1.778" layer="96" rot="R180"/>
@@
 <instance part="U15" gate="G$1" x="251.46" y="-119.38"/>
 <instance part="R11" gate="G$1" x="226.06" y="-111.76"/>
-<instance part="R12" gate="G$1" x="342.9" y="-139.7" rot="R90"/>
+<instance part="R19" gate="G$1" x="342.9" y="-139.7" rot="R90"/>
 <instance part="+3V17" gate="G$1" x="335.28" y="-124.46" smashed="yes">
 <attribute name="VALUE" x="332.74" y="-124.46" size="1.778" layer="96" rot="R180"/>
@@
 <wire x1="375.92" y1="-132.08" x2="378.46" y2="-132.08" width="0.1524" layer="91"/>
 <wire x1="378.46" y1="-132.08" x2="378.46" y2="-147.32" width="0.1524" layer="91"/>
-<pinref part="R12" gate="G$1" pin="1"/>
+<pinref part="R19" gate="G$1" pin="1"/>
 <wire x1="342.9" y1="-144.78" x2="342.9" y2="-147.32" width="0.1524" layer="91"/>
 <junction x="342.9" y="-147.32"/>
@@
 <pinref part="U11" gate="G$1" pin="NFAULT"/>
 <wire x1="297.18" y1="-93.98" x2="269.24" y2="-93.98" width="0.1524" layer="91"/>
-<pinref part="R14" gate="G$1" pin="2"/>
+<pinref part="R12" gate="G$1" pin="2"/>
 <wire x1="269.24" y1="-93.98" x2="269.24" y2="-88.9" width="0.1524" layer="91"/>
 <label x="266.7" y="-93.98" size="1.016" layer="95" rot="R180" xref="yes"/>
@@
 <pinref part="P+4" gate="1" pin="+5V"/>
 <wire x1="373.38" y1="-78.74" x2="373.38" y2="-101.6" width="0.1524" layer="91"/>
-<pinref part="R17" gate="G$1" pin="2"/>
+<pinref part="R14" gate="G$1" pin="2"/>
 <wire x1="347.98" y1="-109.22" x2="358.14" y2="-109.22" width="0.1524" layer="91"/>
 <wire x1="358.14" y1="-109.22" x2="358.14" y2="-111.76" width="0.1524" layer="91"/>
 <wire x1="358.14" y1="-111.76" x2="373.38" y2="-111.76" width="0.1524" layer="91"/>
 <wire x1="373.38" y1="-111.76" x2="373.38" y2="-101.6" width="0.1524" layer="91"/>
-<pinref part="R18" gate="G$1" pin="2"/>
+<pinref part="R15" gate="G$1" pin="2"/>
 <wire x1="355.6" y1="-114.3" x2="373.38" y2="-114.3" width="0.1524" layer="91"/>
 <wire x1="373.38" y1="-114.3" x2="373.38" y2="-111.76" width="0.1524" layer="91"/>
 <junction x="373.38" y="-111.76"/>
-<pinref part="R16" gate="G$1" pin="2"/>
+<pinref part="R13" gate="G$1" pin="2"/>
 <wire x1="358.14" y1="-101.6" x2="373.38" y2="-101.6" width="0.1524" layer="91"/>
 <junction x="373.38" y="-101.6"/>
@@
 </segment>
 <segment>
-<pinref part="R14" gate="G$1" pin="1"/>
+<pinref part="R12" gate="G$1" pin="1"/>
 <pinref part="P+5" gate="1" pin="+5V"/>
 <wire x1="259.08" y1="-83.82" x2="259.08" y2="-88.9" width="0.1524" layer="91"/>
@@
 <junction x="330.2" y="-149.86"/>
 <pinref part="P+6" gate="1" pin="+5V"/>
-<pinref part="R19" gate="G$1" pin="2"/>
+<pinref part="R18" gate="G$1" pin="2"/>
 <wire x1="330.2" y1="-149.86" x2="330.2" y2="-152.4" width="0.1524" layer="91"/>
 <junction x="330.2" y="-152.4"/>
 <wire x1="330.2" y1="-152.4" x2="330.2" y2="-157.48" width="0.1524" layer="91"/>
-<pinref part="R20" gate="G$1" pin="2"/>
-<pinref part="R21" gate="G$1" pin="2"/>
+<pinref part="R17" gate="G$1" pin="2"/>
+<pinref part="R16" gate="G$1" pin="2"/>
 <wire x1="342.9" y1="-175.26" x2="335.28" y2="-175.26" width="0.1524" layer="91"/>
 <wire x1="335.28" y1="-175.26" x2="330.2" y2="-175.26" width="0.1524" layer="91"/>
@@
 <wire x1="327.66" y1="-101.6" x2="337.82" y2="-101.6" width="0.1524" layer="91"/>
 <wire x1="337.82" y1="-101.6" x2="337.82" y2="-109.22" width="0.1524" layer="91"/>
-<pinref part="R17" gate="G$1" pin="1"/>
+<pinref part="R14" gate="G$1" pin="1"/>
 </segment>
 </net>
@@
 <pinref part="U11" gate="G$1" pin="DEC1"/>
 <wire x1="327.66" y1="-106.68" x2="330.2" y2="-106.68" width="0.1524" layer="91"/>
-<pinref part="R18" gate="G$1" pin="1"/>
+<pinref part="R15" gate="G$1" pin="1"/>
 <wire x1="330.2" y1="-106.68" x2="330.2" y2="-114.3" width="0.1524" layer="91"/>
 <wire x1="330.2" y1="-114.3" x2="345.44" y2="-114.3" width="0.1524" layer="91"/>
@@
 <pinref part="U11" gate="G$1" pin="ADEC"/>
 <wire x1="327.66" y1="-93.98" x2="347.98" y2="-93.98" width="0.1524" layer="91"/>
-<pinref part="R16" gate="G$1" pin="1"/>
+<pinref part="R13" gate="G$1" pin="1"/>
 <wire x1="347.98" y1="-93.98" x2="347.98" y2="-101.6" width="0.1524" layer="91"/>
 </segment>
@@
 <wire x1="342.9" y1="-160.02" x2="342.9" y2="-165.1" width="0.1524" layer="91"/>
 <junction x="342.9" y="-160.02"/>
-<pinref part="R20" gate="G$1" pin="1"/>
+<pinref part="R17" gate="G$1" pin="1"/>
 <pinref part="U13" gate="G$1" pin="SDA2"/>
 </segment>
@@
 <wire x1="335.28" y1="-162.56" x2="335.28" y2="-165.1" width="0.1524" layer="91"/>
 <junction x="335.28" y="-162.56"/>
-<pinref part="R21" gate="G$1" pin="1"/>
+<pinref part="R16" gate="G$1" pin="1"/>
 <pinref part="U13" gate="G$1" pin="SCL2"/>
 </segment>
@@
 <pinref part="U13" gate="G$1" pin="EN"/>
 <pinref part="U13" gate="G$1" pin="VREF2"/>
-<pinref part="R19" gate="G$1" pin="1"/>
+<pinref part="R18" gate="G$1" pin="1"/>
 <wire x1="342.9" y1="-152.4" x2="345.44" y2="-152.4" width="0.1524" layer="91"/>
 <wire x1="345.44" y1="-152.4" x2="345.44" y2="-157.48" width="0.1524" layer="91"/>
@@
 <pinref part="U14" gate="G$1" pin="!OE!"/>
 <wire x1="345.44" y1="-132.08" x2="342.9" y2="-132.08" width="0.1524" layer="91"/>
-<pinref part="R12" gate="G$1" pin="2"/>
+<pinref part="R19" gate="G$1" pin="2"/>
 <wire x1="342.9" y1="-132.08" x2="342.9" y2="-134.62" width="0.1524" layer="91"/>
 </segment>

Commit message: Did a bunch of stuff: Swapped to larger onboard flash (128 MB), Added debug UART, Removed pressure senaor and replaced with header to external board, moved each comm interface to use only one SERCOM.
Parts:
- removed U5: HSCMNNN1.6BAAA3, NR_IC:HSCMNNN1.6BAAA3
- added JP6: (no value), pinhead:PINHD-1X3
- added JP7: (no value), pinhead:PINHD-1X5
- added R20: 4.7k, resistor:R-US_R0603
- U8: value S25FL127SABMFI101 -> MT25QL01GBBB8ESF-0AAT; device NR_IC:S25FL127SABMFI101 -> NR_IC:MT25QL01GBBB8ESF-0AAT
Connections:
- removed net PA24: U1.PA24/EIC/SCOM3PAD2+/TC5, U3.INT1
- removed net PA25: U1.PA25/EIC/SCOM3PAD3+/TC5, U3.INT2
- new net N$32: R20.2, U8.!RESET!, U8.DQ3/!HOLD!
- new net PB02: U1.PB02/EIC/AIN10/SCOM5PAD0, U3.INT1
- new net PB03: U1.PB03/EIC/AIN11/SCOM5PAD1, U3.INT2
- new net RX2: JP6.2, U1.PA25/EIC/SCOM3PAD3+/TC5
- new net TX2: JP6.1, U1.PA24/EIC/SCOM3PAD2+/TC5
- net +3V3: now also JP7.1, R20.1; no longer U5.VS
- net GND: now also JP6.3, JP7.5, U8.VSS; no longer U5.GND, U8.GND
- net MISO: now also U1.PB09/EIC/AIN3/SCOM4PAD1//TC4, U8.DQ1; no longer U1.PA12/I2C/EIC/SCOM2PAD0+/TC2, U8.SO/IO1
- net MOSI: now also U8.DQ0; no longer U8.SI/IO0
- net PA06: now also JP7.4; no longer U5.VOUT
- net PB23: now also U8.!S!; no longer U8.!CS!
- net SCK: now also U8.C; no longer U8.CLK
- net SCL: now also JP7.3
- net SDA: now also JP7.2
Other:
- note added: "CARRIER BOARD IO"
- note added: "DEBUG UART"
- note removed: "PRESSURE SENSE"
- moved on the sheet: C15, C16, C17, C23, U3

Commit message: Updated Motor Driver Configuration
Made motor driver decay mode configurable via the multiplexer
Changed current sense resistors to 1.05 ohm for more granular control
over current limiting
Added a pull-up on nENBL so the output stage will be disabled until
explicitly commanded otherwise
Renumbered resistors accordingly
Parts:
- removed R19: 10k, rcl:R-US_R0603
- R10, R9: value 560m -> 1.05
- R15: value 10k -> 4.7k
- R17: value 4.7k -> 220k
- R18: value 220k -> 10k
Connections:
- removed net N$17: R14.1, U11.DEC0
- removed net N$18: R15.1, U11.DEC1
- new net DEC0: U10.P10, U11.DEC0
- new net DEC1: U10.P11, U11.DEC1
- net +5V: now also R14.1; no longer R14.2, R18.2
- net GND: now also R18.1; no longer R19.1
- net N$27: now also R18.2; no longer R19.2
- net N$33: now also R16.1; no longer R17.1
- net N$34: now also R15.1; no longer R16.1
- net N$35: now also R17.1; no longer R18.1
- net NENBL: now also R14.2, U10.P07; no longer U10.P11
- net NSLEEP: now also U10.P06; no longer U10.P10
Other:
- moved on the sheet: R13, R14, R15, R16, R17, R18

Commit message: added gitignore, updated schematic for analog reference and LED driver PWM
Connections:
- net PA09 renamed LED_CTRL
- removed net VREFA_IN: L4.2
- net +3V3: now also L4.2
Changed lines of the file:
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@@
 <?xml version="1.0" encoding="utf-8"?>
 <!DOCTYPE eagle SYSTEM "eagle.dtd">
-<eagle version="7.5.0">
+<eagle version="7.7.0">
 <drawing>
 <settings>
@@
 <part name="JP7" library="pinhead" deviceset="PINHD-1X5" device=""/>
 <part name="R14" library="rcl" deviceset="R-US_" device="R0603" value="10k"/>
+<part name="+3V18" library="supply1" deviceset="+3V3" device=""/>
 </parts>
 <sheets>
@@
 <instance part="JP7" gate="A" x="358.14" y="99.06"/>
 <instance part="R14" gate="G$1" x="266.7" y="-99.06"/>
+<instance part="+3V18" gate="G$1" x="287.02" y="111.76" smashed="yes" rot="R270">
+<attribute name="VALUE" x="281.94" y="114.3" size="1.778" layer="96"/>
+</instance>
 </instances>
 <busses>
@@
 <wire x1="345.44" y1="104.14" x2="355.6" y2="104.14" width="0.1524" layer="91"/>
 </segment>
+<segment>
+<wire x1="279.4" y1="111.76" x2="284.48" y2="111.76" width="0.1524" layer="91"/>
+<pinref part="L4" gate="G$1" pin="2"/>
+<pinref part="+3V18" gate="G$1" pin="+3V3"/>
+</segment>
 </net>
 <net name="GND" class="0">
@@
 </segment>
 </net>
-<net name="PA09" class="0">
-<segment>
-<pinref part="U1" gate="G$1" pin="PA09/I2C/EIC/AIN17/SCOM2PAD1+/TC0"/>
-<wire x1="152.4" y1="86.36" x2="185.42" y2="86.36" width="0.1524" layer="91"/>
-<label x="185.42" y="86.36" size="1.016" layer="95" xref="yes"/>
-</segment>
-<segment>
-<pinref part="U9" gate="G$1" pin="EN"/>
-<wire x1="-111.76" y1="-78.74" x2="-132.08" y2="-78.74" width="0.1524" layer="91"/>
-<label x="-132.08" y="-78.74" size="1.016" layer="95" rot="R180" xref="yes"/>
-</segment>
-</net>
 <net name="MISO" class="0">
 <segment>
@@
 <wire x1="93.98" y1="-30.48" x2="104.14" y2="-30.48" width="0.1524" layer="91"/>
 <label x="104.14" y="-30.48" size="1.016" layer="95" xref="yes"/>
-</segment>
-</net>
-<net name="VREFA_IN" class="0">
-<segment>
-<wire x1="279.4" y1="111.76" x2="284.48" y2="111.76" width="0.1524" layer="91"/>
-<label x="284.48" y="111.76" size="1.016" layer="95" xref="yes"/>
-<pinref part="L4" gate="G$1" pin="2"/>
 </segment>
 </net>
@@
 </segment>
 </net>
+<net name="LED_CTRL" class="0">
+<segment>
+<pinref part="U9" gate="G$1" pin="EN"/>
+<wire x1="-111.76" y1="-78.74" x2="-132.08" y2="-78.74" width="0.1524" layer="91"/>
+<label x="-132.08" y="-78.74" size="1.016" layer="95" rot="R180" xref="yes"/>
+</segment>
+<segment>
+<pinref part="U1" gate="G$1" pin="PA09/I2C/EIC/AIN17/SCOM2PAD1+/TC0"/>
+<wire x1="152.4" y1="86.36" x2="185.42" y2="86.36" width="0.1524" layer="91"/>
+<label x="185.42" y="86.36" size="1.016" layer="95" xref="yes"/>
+</segment>
+</net>

Commit message: Stuff
Parts:
- removed C10, C13: 100nF, resistor:C-USC0603
- removed C14: 1nF, resistor:C-USC0603
- removed L5: 10uH, AR_passives:INDUCTOR-0603
- removed U2: ACS722LLCTR-10AU, NR_IC:ACS722LLCTR-10AU
Connections:
- removed net PA05: C14.1, U1.PA05/EIC/AIN5/SCOM0PAD1, U2.VIOUT
- removed net PA07: U1.PA07/EIC/AIN7/SCOM0PAD3
- removed net VREFB: C10.1, L5.1, U1.PA04/EIC/REF/AIN4/SCOM0PAD0/VREFB
- removed net VREFB_IN: L5.2
- removed net V_UNREG: U2.IP-@1, U2.IP-@2
- new net I_SENSE: U1.PA05/EIC/AIN5/SCOM0PAD1
- new net USB_D+: U1.PA25/EIC/SCOM3PAD3+/TC5
- new net USB_D-: U1.PA24/EIC/SCOM3PAD2+/TC5
- net +3V3: no longer C13.1, U2.VCC
- net +5V: no longer U2.IP+@1, U2.IP+@2
- net GND: no longer C10.2, C13.2, C14.2, U2.BW_SEL, U2.GND
- net RX2: now also U1.PA07/EIC/AIN7/SCOM0PAD3; no longer U1.PA25/EIC/SCOM3PAD3+/TC5
- net TX2: now also U1.PA04/EIC/REF/AIN4/SCOM0PAD0/VREFB; no longer U1.PA24/EIC/SCOM3PAD2+/TC5
Other:
- note removed: "I SENSE"
- moved on the sheet: C9, L4

Commit message: Renamed some nets, reorganized a bit, removed unnecessary headers
Parts:
- removed JP2, JP3, JP6: (no value), pinhead:PINHD-1X3
- removed JP4: (no value), NR_Pinhead:SCREWTERM_1X2
- removed JP5: (no value), pinhead:PINHD-1X4
- removed JP7: (no value), pinhead:PINHD-1X5
Connections:
- removed net PA06: JP7.4, U1.PA06/EIC/AIN6/SCOM0PAD2
- removed net PA13: U1.PA13/I2C/EIC/SCOM2PAD1+/TC2
- new net PRESSURE_IN: U1.PA06/EIC/AIN6/SCOM0PAD2
- new net SYNC: U1.PA12/I2C/EIC/SCOM2PAD0+/TC2
- net +3V3: no longer JP7.1
- net GND: no longer JP2.3, JP3.3, JP6.3, JP7.5
- net LED_GND: no longer JP4.1
- net LED_V: no longer JP4.2
- net MA1: no longer JP5.1
- net MA2: no longer JP5.2
- net MB1: no longer JP5.3
- net MB2: no longer JP5.4
- net RX0: no longer JP2.2
- net RX1: no longer JP3.2
- net RX2: no longer JP6.2
- net SCL: no longer JP7.3
- net SDA: no longer JP7.2
- net TX0: no longer JP2.1
- net TX1: no longer JP3.1
- net TX2: no longer JP6.1
Other:
- note removed: "CARRIER BOARD IO"
- note removed: "DEBUG UART"
- note removed: "UART CTU"
- note removed: "UART PI ZERO"
