File: CAD/eagle/STARduino/starduino.sch (EAGLE design)
At the start: 123 parts, among them J1 J30J-9J30, J2 MICRO_SD, J3 J30J-15J30, J4 J30J-31J30, J5 RPI-ZERO, J6 RPI-CSI, Q1 FDG8842CZ, Q2 FDG8842CZ, Q3 DMMT5401, Q4 DMG2305UX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

Commit message: layout stuff
Connections:
- net IMUDR: now also U9.DIN; no longer U9.AIN
- net IMUINT3: now also U9.AIN; no longer U9.DIN
Changed lines of the file:
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@@
 <?xml version="1.0" encoding="utf-8"?>
 <!DOCTYPE eagle SYSTEM "eagle.dtd">
-<eagle version="7.7.0">
+<eagle version="6.5.0">
 <drawing>
 <settings>
@@
 </segment>
 <segment>
+<wire x1="396.24" y1="139.7" x2="393.7" y2="139.7" width="0.1524" layer="91"/>
+<label x="393.7" y="139.7" size="1.016" layer="95" rot="R180" xref="yes"/>
+<pinref part="U9" gate="G$1" pin="DIN"/>
+</segment>
+</net>
+<net name="IMUINT1" class="0">
+<segment>
+<label x="497.84" y="254" size="1.016" layer="95" xref="yes"/>
+<pinref part="U13" gate="G$1" pin="INT1"/>
+<wire x1="485.14" y1="254" x2="497.84" y2="254" width="0.1524" layer="91"/>
+</segment>
+<segment>
+<wire x1="396.24" y1="144.78" x2="393.7" y2="144.78" width="0.1524" layer="91"/>
+<label x="393.7" y="144.78" size="1.016" layer="95" rot="R180" xref="yes"/>
+<pinref part="U9" gate="G$1" pin="BIN"/>
+</segment>
+</net>
+<net name="IMUINT2" class="0">
+<segment>
+<label x="497.84" y="251.46" size="1.016" layer="95" xref="yes"/>
+<pinref part="U13" gate="G$1" pin="INT2"/>
+<wire x1="485.14" y1="251.46" x2="497.84" y2="251.46" width="0.1524" layer="91"/>
+</segment>
+<segment>
+<wire x1="396.24" y1="142.24" x2="393.7" y2="142.24" width="0.1524" layer="91"/>
+<label x="393.7" y="142.24" size="1.016" layer="95" rot="R180" xref="yes"/>
+<pinref part="U9" gate="G$1" pin="CIN"/>
+</segment>
+</net>
+<net name="IMUINT3" class="0">
+<segment>
+<label x="497.84" y="248.92" size="1.016" layer="95" xref="yes"/>
+<pinref part="U13" gate="G$1" pin="INT3"/>
+<wire x1="485.14" y1="248.92" x2="497.84" y2="248.92" width="0.1524" layer="91"/>
+</segment>
+<segment>
 <wire x1="396.24" y1="147.32" x2="393.7" y2="147.32" width="0.1524" layer="91"/>
 <label x="393.7" y="147.32" size="1.016" layer="95" rot="R180" xref="yes"/>
@@
 </segment>
 </net>
-<net name="IMUINT1" class="0">
-<segment>
-<label x="497.84" y="254" size="1.016" layer="95" xref="yes"/>
-<pinref part="U13" gate="G$1" pin="INT1"/>
-<wire x1="485.14" y1="254" x2="497.84" y2="254" width="0.1524" layer="91"/>
-</segment>
-<segment>
-<wire x1="396.24" y1="144.78" x2="393.7" y2="144.78" width="0.1524" layer="91"/>
-<label x="393.7" y="144.78" size="1.016" layer="95" rot="R180" xref="yes"/>
-<pinref part="U9" gate="G$1" pin="BIN"/>
-</segment>
-</net>
-<net name="IMUINT2" class="0">
-<segment>
-<label x="497.84" y="251.46" size="1.016" layer="95" xref="yes"/>
-<pinref part="U13" gate="G$1" pin="INT2"/>
-<wire x1="485.14" y1="251.46" x2="497.84" y2="251.46" width="0.1524" layer="91"/>
-</segment>
-<segment>
-<wire x1="396.24" y1="142.24" x2="393.7" y2="142.24" width="0.1524" layer="91"/>
-<label x="393.7" y="142.24" size="1.016" layer="95" rot="R180" xref="yes"/>
-<pinref part="U9" gate="G$1" pin="CIN"/>
-</segment>
-</net>
-<net name="IMUINT3" class="0">
-<segment>
-<label x="497.84" y="248.92" size="1.016" layer="95" xref="yes"/>
-<pinref part="U13" gate="G$1" pin="INT3"/>
-<wire x1="485.14" y1="248.92" x2="497.84" y2="248.92" width="0.1524" layer="91"/>
-</segment>
-<segment>
-<wire x1="396.24" y1="139.7" x2="393.7" y2="139.7" width="0.1524" layer="91"/>
-<label x="393.7" y="139.7" size="1.016" layer="95" rot="R180" xref="yes"/>
-<pinref part="U9" gate="G$1" pin="DIN"/>
-</segment>
-</net>

Commit message: stuff
Parts:
- removed C28: 1μF, resistor:C-USC0603
- removed F1: 1206L150THWR, adafruit:PTCFUSE-1206
- removed Q3: DMMT5401, transistor-pnp:DMMT5401
- removed Q4: DMG2305UX, microbuilder:MOSFET-P
- removed R15: 10k, resistor:R-US_R0603
- removed R16: 47k, resistor:R-US_R0603
Connections:
- removed net N$53: J5.5V, Q3.E2, Q4.D
- removed net N$54: Q3.C2, Q4.G, R16.1
- removed net N$55: Q3.B1, Q3.B2, Q3.C1, R15.1
- removed net N$56: C28.1, F1.2, Q3.E1, Q4.S
- net +5V: no longer F1.1
- net GND: no longer C28.2, R15.2, R16.2
- net PI_5V: now also J5.5V
Changed lines of the file:
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@@
 <part name="GND52" library="supply1" deviceset="GND" device=""/>
 <part name="GND53" library="supply1" deviceset="GND" device=""/>
-<part name="Q3" library="transistor-pnp" deviceset="DMMT5401" device=""/>
-<part name="Q4" library="microbuilder" deviceset="MOSFET-P" device="" value="DMG2305UX"/>
-<part name="F1" library="adafruit" deviceset="PTCFUSE" device="-1206" value="1206L150THWR"/>
-<part name="R16" library="resistor" deviceset="R-US_" device="R0603" value="47k"/>
-<part name="R15" library="resistor" deviceset="R-US_" device="R0603" value="10k"/>
-<part name="GND54" library="SparkFun-Aesthetics" deviceset="GND" device=""/>
-<part name="GND55" library="SparkFun-Aesthetics" deviceset="GND" device=""/>
-<part name="C28" library="resistor" deviceset="C-US" device="C0603" value="1μF"/>
-<part name="GND56" library="SparkFun-Aesthetics" deviceset="GND" device=""/>
 <part name="J5" library="CM_connectors" deviceset="RPI-ZERO" device=""/>
-<part name="P+15" library="supply1" deviceset="+5V" device=""/>
 <part name="GND57" library="SparkFun-Aesthetics" deviceset="GND" device=""/>
 <part name="J6" library="CM_connectors" deviceset="RPI-CSI" device=""/>
@@
 <instance part="GND52" gate="1" x="208.28" y="114.3"/>
 <instance part="GND53" gate="1" x="195.58" y="88.9"/>
-<instance part="Q3" gate="G$1" x="284.48" y="134.62"/>
-<instance part="Q4" gate="G$1" x="287.02" y="147.32" rot="R90"/>
-<instance part="F1" gate="G$1" x="266.7" y="149.86"/>
-<instance part="R16" gate="G$1" x="294.64" y="116.84" rot="R270"/>
-<instance part="R15" gate="G$1" x="279.4" y="116.84" rot="R270"/>
-<instance part="GND54" gate="1" x="294.64" y="106.68"/>
-<instance part="GND55" gate="1" x="279.4" y="106.68"/>
-<instance part="C28" gate="G$1" x="271.78" y="144.78"/>
-<instance part="GND56" gate="1" x="271.78" y="134.62"/>
 <instance part="J5" gate="G$1" x="340.36" y="119.38"/>
-<instance part="P+15" gate="1" x="261.62" y="160.02" smashed="yes">
-<attribute name="VALUE" x="269.24" y="160.02" size="1.778" layer="96" rot="R180"/>
-</instance>
 <instance part="GND57" gate="1" x="314.96" y="83.82"/>
 <instance part="J6" gate="G$1" x="347.98" y="193.04"/>
@@
 <pinref part="GND53" gate="1" pin="GND"/>
 <wire x1="215.9" y1="91.44" x2="195.58" y2="91.44" width="0.1524" layer="91"/>
-</segment>
-<segment>
-<pinref part="GND54" gate="1" pin="GND"/>
-<pinref part="R16" gate="G$1" pin="2"/>
-<wire x1="294.64" y1="109.22" x2="294.64" y2="111.76" width="0.1524" layer="91"/>
-</segment>
-<segment>
-<pinref part="R15" gate="G$1" pin="2"/>
-<pinref part="GND55" gate="1" pin="GND"/>
-<wire x1="279.4" y1="111.76" x2="279.4" y2="109.22" width="0.1524" layer="91"/>
-</segment>
-<segment>
-<pinref part="C28" gate="G$1" pin="2"/>
-<pinref part="GND56" gate="1" pin="GND"/>
-<wire x1="271.78" y1="139.7" x2="271.78" y2="137.16" width="0.1524" layer="91"/>
 </segment>
 <segment>
@@
 <wire x1="149.86" y1="99.06" x2="149.86" y2="101.6" width="0.1524" layer="91"/>
 </segment>
-<segment>
-<pinref part="F1" gate="G$1" pin="1"/>
-<wire x1="261.62" y1="152.4" x2="261.62" y2="157.48" width="0.1524" layer="91"/>
-<pinref part="P+15" gate="1" pin="+5V"/>
-</segment>
 </net>
 <net name="LED_GND" class="0">
@@
 <wire x1="152.4" y1="193.04" x2="154.94" y2="193.04" width="0.1524" layer="91"/>
 <label x="154.94" y="193.04" size="1.016" layer="95" xref="yes"/>
+</segment>
+<segment>
+<pinref part="J5" gate="G$1" pin="5V"/>
+<wire x1="317.5" y1="147.32" x2="312.42" y2="147.32" width="0.1524" layer="91"/>
+<label x="312.42" y="147.32" size="1.016" layer="95" rot="R180" xref="yes"/>
 </segment>
 </net>
@@
 </segment>
 </net>
-<net name="N$53" class="0">
-<segment>
-<pinref part="Q3" gate="G$1" pin="E2"/>
-<wire x1="294.64" y1="147.32" x2="294.64" y2="142.24" width="0.1524" layer="91"/>
-<pinref part="Q4" gate="G$1" pin="D"/>
-<wire x1="294.64" y1="147.32" x2="292.1" y2="147.32" width="0.1524" layer="91"/>
-<junction x="294.64" y="147.32"/>
-<wire x1="294.64" y1="147.32" x2="317.5" y2="147.32" width="0.1524" layer="91"/>
-<pinref part="J5" gate="G$1" pin="5V"/>
-</segment>
-</net>
-<net name="N$54" class="0">
-<segment>
-<pinref part="Q3" gate="G$1" pin="C2"/>
-<pinref part="R16" gate="G$1" pin="1"/>
-<wire x1="294.64" y1="127" x2="294.64" y2="124.46" width="0.1524" layer="91"/>
-<pinref part="Q4" gate="G$1" pin="G"/>
-<wire x1="294.64" y1="124.46" x2="294.64" y2="121.92" width="0.1524" layer="91"/>
-<wire x1="284.48" y1="142.24" x2="302.26" y2="142.24" width="0.1524" layer="91"/>
-<wire x1="302.26" y1="142.24" x2="302.26" y2="124.46" width="0.1524" layer="91"/>
-<wire x1="302.26" y1="124.46" x2="294.64" y2="124.46" width="0.1524" layer="91"/>
-<junction x="294.64" y="124.46"/>
-</segment>
-</net>
-<net name="N$55" class="0">
-<segment>
-<pinref part="Q3" gate="G$1" pin="B2"/>
-<wire x1="289.56" y1="127" x2="289.56" y2="124.46" width="0.1524" layer="91"/>
-<wire x1="289.56" y1="124.46" x2="284.48" y2="124.46" width="0.1524" layer="91"/>
-<pinref part="Q3" gate="G$1" pin="C1"/>
-<wire x1="284.48" y1="124.46" x2="279.4" y2="124.46" width="0.1524" layer="91"/>
-<wire x1="279.4" y1="124.46" x2="279.4" y2="127" width="0.1524" layer="91"/>
-<pinref part="Q3" gate="G$1" pin="B1"/>
-<wire x1="284.48" y1="127" x2="284.48" y2="124.46" width="0.1524" layer="91"/>
-<junction x="284.48" y="124.46"/>
-<pinref part="R15" gate="G$1" pin="1"/>
-<wire x1="279.4" y1="124.46" x2="279.4" y2="121.92" width="0.1524" layer="91"/>
-<junction x="279.4" y="124.46"/>
-</segment>
-</net>
-<net name="N$56" class="0">
-<segment>
-<pinref part="Q4" gate="G$1" pin="S"/>
-<pinref part="Q3" gate="G$1" pin="E1"/>
-<wire x1="281.94" y1="147.32" x2="279.4" y2="147.32" width="0.1524" layer="91"/>
-<wire x1="279.4" y1="147.32" x2="279.4" y2="142.24" width="0.1524" layer="91"/>
-<pinref part="C28" gate="G$1" pin="1"/>
-<wire x1="279.4" y1="147.32" x2="271.78" y2="147.32" width="0.1524" layer="91"/>
-<junction x="279.4" y="147.32"/>
-<pinref part="F1" gate="G$1" pin="2"/>
-<wire x1="271.78" y1="147.32" x2="271.78" y2="152.4" width="0.1524" layer="91"/>
-<junction x="271.78" y="147.32"/>
-</segment>
-</net>
