File: CAD/eagle/STARduino/starduino.sch (EAGLE design)
At the start: 117 parts, among them J1 J30J-9J30, J2 MICRO_SD, J3 J30J-15J30, J4 J30J-31J30, J5 RPI-ZERO, J6 RPI-CSI, Q1 FDG8842CZ, Q2 FDG8842CZ, Q5 FDG8842CZ, Q6 FDG8842CZ, T1 750313972, U1 LT8301, U10 MC74VHC1GT125DT, U11 TCA9535_RTW_24, U12 MAX31725MTA+, U13 BMX055, U14 DRV8846RGER, U15 P82B715, U16 MC74VHC1GT125DT, U17 PCA9306DCT, U2 LT3465/A, U3 LTC3112FE, U4 DS3231MZ+, U5 MT25QL01GBBB8ESF-0AAT, U6 ATSAMD21G18, U7 MIC5216, U8 ADXL375BCCZ, U9 MC14504BDTG

Commit message: Package stuff
Connections:
- removed net USB_D+: U6.PA25/EIC/SCOM3PAD3+/TC5
- removed net USB_D-: U6.PA24/EIC/SCOM3PAD2+/TC5
- net USB_D_N: now also U6.PA24/EIC/SCOM3PAD2+/TC5
- net USB_D_P: now also U6.PA25/EIC/SCOM3PAD3+/TC5
Changed lines of the file:
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@@
-</segment>
-</net>
-<net name="USB_D-" class="0">
-<segment>
-<pinref part="U6" gate="G$1" pin="PA24/EIC/SCOM3PAD2+/TC5"/>
-<wire x1="312.42" y1="342.9" x2="345.44" y2="342.9" width="0.1524" layer="91"/>
-<label x="345.44" y="342.9" size="1.016" layer="95" xref="yes"/>
-</segment>
-</net>
-<net name="USB_D+" class="0">
-<segment>
-<pinref part="U6" gate="G$1" pin="PA25/EIC/SCOM3PAD3+/TC5"/>
-<wire x1="312.42" y1="340.36" x2="345.44" y2="340.36" width="0.1524" layer="91"/>
-<label x="345.44" y="340.36" size="1.016" layer="95" xref="yes"/>
 </segment>
 </net>
@@
 <label x="162.56" y="109.22" size="1.016" layer="95" rot="R180" xref="yes"/>
 </segment>
+<segment>
+<pinref part="U6" gate="G$1" pin="PA25/EIC/SCOM3PAD3+/TC5"/>
+<wire x1="312.42" y1="340.36" x2="345.44" y2="340.36" width="0.1524" layer="91"/>
+<label x="345.44" y="340.36" size="1.016" layer="95" xref="yes"/>
+</segment>
 </net>
 <net name="USB_D_N" class="0">
@@
 <label x="162.56" y="104.14" size="1.016" layer="95" rot="R180" xref="yes"/>
 </segment>
-</net>
+<segment>
+<pinref part="U6" gate="G$1" pin="PA24/EIC/SCOM3PAD2+/TC5"/>
+<wire x1="312.42" y1="342.9" x2="345.44" y2="342.9" width="0.1524" layer="91"/>
+<label x="345.44" y="342.9" size="1.016" layer="95" xref="yes"/>
+</segment>
+</net>

Commit message: layout stuff
Parts:
- TP1, TP2: value TESTPOINT -> TESTPOINT1.5MM; device CM_passives:TESTPOINT -> CM_passives:TESTPOINT1.5MM
- U10, U16: value MC74VHC1GT125DT -> MC74VHC1GT125; device MotorDriver:MC74VHC1GT125DT -> CM_IC:MC74VHC1GT125
Connections:
- net +3V3: now also U16.VIN; no longer U16.VCC
- net +5V: now also U10.VIN; no longer U10.VCC
- net GND: now also U10.OE, U16.OE; no longer U10.!OE!, U16.!OE!
- net IOEINT: now also U16.Y; no longer U16.OUTY
- net N$22: now also U10.Y; no longer U10.OUTY
- net N$25: now also U16.A; no longer U16.INA
- net PI_D_N: now also J3.7; no longer J3.8
- net PI_D_P: now also J3.8; no longer J3.7
- net STEPFREQ: now also U10.A; no longer U10.INA
Changed lines of the file:
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@@
 <part name="+3V16" library="supply1" deviceset="+3V3" device=""/>
 <part name="U17" library="MotorDriver" deviceset="PCA9306" device="DCT"/>
-<part name="U16" library="MotorDriver" deviceset="MC74VHC1GT125" device="DT"/>
-<part name="U10" library="MotorDriver" deviceset="MC74VHC1GT125" device="DT"/>
+<part name="U16" library="CM_IC" deviceset="MC74VHC1GT125" device=""/>
+<part name="U10" library="CM_IC" deviceset="MC74VHC1GT125" device=""/>
 <part name="+3V17" library="supply1" deviceset="+3V3" device=""/>
 <part name="U5" library="NR_IC" deviceset="MT25QL01GBBB8ESF-0AAT" device=""/>
@@
 <part name="GND58" library="supply1" deviceset="GND" device=""/>
 <part name="GND59" library="supply1" deviceset="GND" device=""/>
-<part name="TP1" library="CM_passives" deviceset="TESTPOINT" device=""/>
-<part name="TP2" library="CM_passives" deviceset="TESTPOINT" device=""/>
+<part name="TP1" library="CM_passives" deviceset="TESTPOINT" device="1.5MM"/>
+<part name="TP2" library="CM_passives" deviceset="TESTPOINT" device="1.5MM"/>
 </parts>
 <sheets>
@@
 </segment>
 <segment>
-<pinref part="U16" gate="G$1" pin="VCC"/>
+<pinref part="U16" gate="G$1" pin="VIN"/>
 <wire x1="513.08" y1="165.1" x2="513.08" y2="167.64" width="0.1524" layer="91"/>
 <pinref part="+3V17" gate="G$1" pin="+3V3"/>
@@
 <wire x1="429.26" y1="175.26" x2="429.26" y2="185.42" width="0.1524" layer="91"/>
 <wire x1="396.24" y1="175.26" x2="396.24" y2="195.58" width="0.1524" layer="91"/>
-<pinref part="U10" gate="G$1" pin="!OE!"/>
+<pinref part="U10" gate="G$1" pin="OE"/>
 <wire x1="396.24" y1="195.58" x2="398.78" y2="195.58" width="0.1524" layer="91"/>
 <pinref part="U10" gate="G$1" pin="GND"/>
@@
 <wire x1="513.08" y1="149.86" x2="513.08" y2="147.32" width="0.1524" layer="91"/>
 <junction x="513.08" y="147.32"/>
-<pinref part="U16" gate="G$1" pin="!OE!"/>
+<pinref part="U16" gate="G$1" pin="OE"/>
 <wire x1="502.92" y1="165.1" x2="495.3" y2="165.1" width="0.1524" layer="91"/>
 <wire x1="495.3" y1="165.1" x2="495.3" y2="147.32" width="0.1524" layer="91"/>
@@
 <wire x1="419.1" y1="205.74" x2="411.48" y2="205.74" width="0.1524" layer="91"/>
 <wire x1="411.48" y1="205.74" x2="408.94" y2="205.74" width="0.1524" layer="91"/>
-<pinref part="U10" gate="G$1" pin="VCC"/>
+<pinref part="U10" gate="G$1" pin="VIN"/>
 <wire x1="408.94" y1="205.74" x2="408.94" y2="195.58" width="0.1524" layer="91"/>
 <wire x1="411.48" y1="210.82" x2="411.48" y2="205.74" width="0.1524" layer="91"/>
@@
 <segment>
 <label x="391.16" y="187.96" size="1.016" layer="95" rot="R180" xref="yes"/>
-<pinref part="U10" gate="G$1" pin="INA"/>
+<pinref part="U10" gate="G$1" pin="A"/>
 <wire x1="398.78" y1="187.96" x2="391.16" y2="187.96" width="0.1524" layer="91"/>
 </segment>
@@
 <segment>
 <label x="528.32" y="157.48" size="1.016" layer="95" xref="yes"/>
-<pinref part="U16" gate="G$1" pin="OUTY"/>
+<pinref part="U16" gate="G$1" pin="Y"/>
 <wire x1="523.24" y1="157.48" x2="528.32" y2="157.48" width="0.1524" layer="91"/>
 </segment>
@@
 <segment>
 <pinref part="U14" gate="G$1" pin="STEP"/>
-<pinref part="U10" gate="G$1" pin="OUTY"/>
+<pinref part="U10" gate="G$1" pin="Y"/>
 <wire x1="457.2" y1="187.96" x2="419.1" y2="187.96" width="0.1524" layer="91"/>
 </segment>
@@
 <wire x1="480.06" y1="139.7" x2="480.06" y2="157.48" width="0.1524" layer="91"/>
 <wire x1="480.06" y1="157.48" x2="502.92" y2="157.48" width="0.1524" layer="91"/>
-<pinref part="U16" gate="G$1" pin="INA"/>
+<pinref part="U16" gate="G$1" pin="A"/>
 </segment>
 </net>
@@
 <net name="PI_D_P" class="0">
 <segment>
+<pinref part="TP1" gate="G$1" pin="P$1"/>
+<wire x1="284.48" y1="96.52" x2="281.94" y2="96.52" width="0.1524" layer="91"/>
+<label x="281.94" y="96.52" size="1.016" layer="95" rot="R180" xref="yes"/>
+</segment>
+<segment>
+<pinref part="J3" gate="G$1" pin="8"/>
+<wire x1="165.1" y1="83.82" x2="162.56" y2="83.82" width="0.1524" layer="91"/>
+<label x="162.56" y="83.82" size="1.016" layer="95" rot="R180" xref="yes"/>
+</segment>
+</net>
+<net name="PI_D_N" class="0">
+<segment>
+<pinref part="TP2" gate="G$1" pin="P$1"/>
+<wire x1="284.48" y1="88.9" x2="281.94" y2="88.9" width="0.1524" layer="91"/>
+<label x="281.94" y="88.9" size="1.016" layer="95" rot="R180" xref="yes"/>
+</segment>
+<segment>
 <pinref part="J3" gate="G$1" pin="7"/>
 <wire x1="165.1" y1="88.9" x2="162.56" y2="88.9" width="0.1524" layer="91"/>
 <label x="162.56" y="88.9" size="1.016" layer="95" rot="R180" xref="yes"/>
 </segment>
-<segment>
-<pinref part="TP1" gate="G$1" pin="P$1"/>
-<wire x1="284.48" y1="96.52" x2="281.94" y2="96.52" width="0.1524" layer="91"/>
-<label x="281.94" y="96.52" size="1.016" layer="95" rot="R180" xref="yes"/>
-</segment>
-</net>
-<net name="PI_D_N" class="0">
-<segment>
-<pinref part="J3" gate="G$1" pin="8"/>
-<wire x1="165.1" y1="83.82" x2="162.56" y2="83.82" width="0.1524" layer="91"/>
-<label x="162.56" y="83.82" size="1.016" layer="95" rot="R180" xref="yes"/>
-</segment>
-<segment>
-<pinref part="TP2" gate="G$1" pin="P$1"/>
-<wire x1="284.48" y1="88.9" x2="281.94" y2="88.9" width="0.1524" layer="91"/>
-<label x="281.94" y="88.9" size="1.016" layer="95" rot="R180" xref="yes"/>
-</segment>
-</net>
+</net>

Commit message: layout progress
Connections:
- removed net PRESSURE_IN: J4.11, U6.PA06/EIC/AIN6/SCOM0PAD2
Changed lines of the file:
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@@
 </variantdefs>
 <classes>
-<class number="0" name="default" width="0.2032" drill="0.381">
+<class number="0" name="default" width="0.1524" drill="0.381">
 <clearance class="0" value="0.1524"/>
 </class>
@@
 </segment>
 </net>
-<net name="PRESSURE_IN" class="0">
-<segment>
-<pinref part="U6" gate="G$1" pin="PA06/EIC/AIN6/SCOM0PAD2"/>
-<wire x1="312.42" y1="388.62" x2="345.44" y2="388.62" width="0.1524" layer="91"/>
-<label x="345.44" y="388.62" size="1.016" layer="95" xref="yes"/>
-</segment>
-<segment>
-<pinref part="J4" gate="G$1" pin="11"/>
-<wire x1="215.9" y1="106.68" x2="213.36" y2="106.68" width="0.1524" layer="91"/>
-<label x="213.36" y="106.68" size="1.016" layer="95" rot="R180" xref="yes"/>
-</segment>
-</net>

Commit message: Final layouts and gerbers
Parts:
- added U$1: SSL.3IN_SILK, images:SSL.3IN_SILK
- added U$2: STAR, images:STAR
- U7: value MIC5216 -> MIC5319; device CM_IC:MIC5216 -> CM_IC:MIC5319
Changed lines of the file:
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@@
 <part name="P+9" library="supply1" deviceset="+5V" device=""/>
 <part name="P+10" library="supply1" deviceset="VCC" device=""/>
-<part name="U7" library="CM_IC" deviceset="MIC5216" device=""/>
+<part name="U7" library="CM_IC" deviceset="MIC5319" device=""/>
 <part name="GND44" library="supply1" deviceset="GND" device=""/>
 <part name="C27" library="resistor" deviceset="C-US" device="C0603" value="1uF"/>
@@
 <part name="TP1" library="CM_passives" deviceset="TESTPOINT" device="1.5MM"/>
 <part name="TP2" library="CM_passives" deviceset="TESTPOINT" device="1.5MM"/>
+<part name="U$1" library="images" deviceset="SSL" device=".3IN_SILK"/>
+<part name="U$2" library="images" deviceset="STAR" device=""/>
 </parts>
 <sheets>
@@
 <instance part="TP1" gate="G$1" x="289.56" y="96.52"/>
 <instance part="TP2" gate="G$1" x="289.56" y="88.9"/>
+<instance part="U$1" gate="G$1" x="546.1" y="48.26"/>
+<instance part="U$2" gate="G$1" x="528.32" y="40.64"/>
 </instances>
 <busses>

Commit message: Adjusted some STARduino things
Parts:
- removed R20, R21, R33, R36: 4.7k, resistor:R-US_R0603
- added C28: 100nF, resistor:C-USC0603
- added R15: 4.7k, SparkFun-Passives:RESISTOR-ARRAY0603-ARV
- C29: value 4.7uF -> 2.2uF; device resistor:CPOL-USA/3216-18R -> resistor:C-USC0603
Connections:
- removed net N$1: L3.2, U6.VCC
- removed net N$2: L4.2, U6.VDDIO1
- removed net N$3: L5.2, U6.VDDIO2
- removed net N$4: FB1.P$2, U6.VDDANA
- new net N$10: C19.1, C20.1, C21.1, C22.1, C23.1, C24.1, FB1.P$2, L3.2, L4.2, L5.2, U6.VCC, U6.VDDANA, U6.VDDIO1, U6.VDDIO2
- new net N$9: C28.1, U7.BYP
- net +3V3: now also C29.1, R15A.2, R15B.2, R15C.2, R15D.2; no longer C19.1, C20.1, C21.1, C22.1, C23.1, C24.1, C29.+, R20.2, R21.2, R33.2, R36.2
- net GND: now also C28.2, C29.2; no longer C29.-
- net SCL: now also R15D.1; no longer R21.1
- net SCL_BUFF: now also R15B.1; no longer R36.1
- net SDA: now also R15C.1; no longer R20.1
- net SDA_BUFF: now also R15A.1; no longer R33.1
Other:
- moved on the sheet: C19, C20, C21, C22, C23, C24, FB1, L3, L4, L5

Commit message: Multiplexer Pinout Change
Small change to multiplexer layout for increased sense-making.
Connections:
- net M0: now also U11.P11; no longer U11.P06
- net NFAULT: now also U11.P06; no longer U11.P11
Changed lines of the file:
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@@
 <?xml version="1.0" encoding="utf-8"?>
 <!DOCTYPE eagle SYSTEM "eagle.dtd">
-<eagle version="6.5.0">
+<eagle version="7.5.0">
 <drawing>
 <settings>
@@
 </segment>
 <segment>
-<pinref part="U11" gate="A" pin="P11"/>
-<wire x1="441.96" y1="121.92" x2="436.88" y2="121.92" width="0.1524" layer="91"/>
-<label x="436.88" y="121.92" size="1.016" layer="95" rot="R180" xref="yes"/>
+<pinref part="U11" gate="A" pin="P06"/>
+<wire x1="441.96" y1="132.08" x2="436.88" y2="132.08" width="0.1524" layer="91"/>
+<label x="436.88" y="132.08" size="1.016" layer="95" rot="R180" xref="yes"/>
 </segment>
 </net>
@@
 </segment>
 <segment>
-<label x="436.88" y="132.08" size="1.016" layer="95" rot="R180" xref="yes"/>
-<pinref part="U11" gate="A" pin="P06"/>
-<wire x1="436.88" y1="132.08" x2="441.96" y2="132.08" width="0.1524" layer="91"/>
-</segment>
-</net>
+<pinref part="U11" gate="A" pin="P11"/>
+<wire x1="441.96" y1="121.92" x2="436.88" y2="121.92" width="0.1524" layer="91"/>
+<label x="436.88" y="121.92" size="1.016" layer="95" rot="R180" xref="yes"/>
+</segment>
+</net>

Commit message: STARduino progress. De-stupified 28V bias
Parts:
- removed C41: 100nF, resistor:C-USC0603
- removed Q5, Q6: FDG8842CZ, NR_Transistor:FDG8842CZ
- removed R30: 220k, rcl:R-US_R0603
- removed R32: 4.7k, rcl:R-US_R0603
- removed R34: 10k, rcl:R-US_R0603
- removed R35: 100k, resistor:R-US_R0603
- removed R37: 191k, resistor:R-US_R0603
- added Q3: BSS8402DW, transistor-fet:BSS8402DW
- added R16: 3.6k, resistor:R-US_R0603
- added R17: 6.8k, resistor:R-US_R0603
- added R20, R21: 1.05, rcl:R-US_R0603
- C17: value 47pF -> 3.3nF; device resistor:C-USC0603 -> resistor:C-USC1206
- C18: value 47uF -> 47pF; device resistor:C-USC1210 -> resistor:C-USC0603
- C19: value 10uF -> 47uF; device resistor:C-USC0603 -> resistor:C-USC1210
- C21, C31, C39: value 100nF -> 10uF
- C26: value 1uF -> 100nF
- C28: value 100nF -> 1uF
- C29: value 2.2uF -> 100nF
- C30, C38: value 10uF -> 2.2uF
- C37: value 2.2uF -> 100nF; device rcl:C-USC0603 -> resistor:C-USC0603
- C40: value 1uF -> 100nF; device resistor:C-USC0603 -> rcl:C-USC0603
- D1: value CMDZ5257B -> CMDZ5248B
- JP1: device pinhead:PINHD-2X3 -> CM_passives:JUMPER-2PTH
- JP2: device CM_passives:JUMPER-2PTH -> pinhead:PINHD-2X3
- Q1, Q2: value FDG8842CZ -> BSS8402DW; device NR_Transistor:FDG8842CZ -> transistor-fet:BSS8402DW
- R10: value 100k -> 10k
- R11: value 191k -> 100k
- R12: value 100k -> 191k
- R13: value 4.7k -> 100k
- R14: value 191k -> 4.7k
- R15: value 4.7k -> 191k; device SparkFun-Passives:RESISTOR-ARRAY0603-ARV -> resistor:R-US_R0603
- R18: value 3.6k -> 10k; device resistor:R-US_R0603 -> rcl:R-US_R0603
- R19: value 6.8k -> 10k; device resistor:R-US_R0603 -> rcl:R-US_R0603
- R2: value 10k -> 130k
- R22: value 10k -> 100k; device rcl:R-US_R0603 -> resistor:R-US_R0603
- R23: value 10k -> 4.7k; device rcl:R-US_R0603 -> resistor:R-US_R0603
- R24: value 1.05 -> 191k; device rcl:R-US_R0603 -> resistor:R-US_R0603
- R25: value 1.05 -> 4.7k
- R26: value 100k -> 220k; device resistor:R-US_R0603 -> rcl:R-US_R0603
- R27: device resistor:R-US_R0603 -> rcl:R-US_R0603
- R28: value 191k -> 4.7k; device resistor:R-US_R0603 -> SparkFun-Passives:RESISTOR-ARRAY0603-ARV
- R29: value 4.7k -> 10k
- R3: value 270k -> 10k
- R7: value 845k -> 1.5k; device resistor:R-US_R0603 -> resistor:R-US_R1206
- R8: value 158k -> 845k
- R9: value 10k -> 158k
- T1: value 750313972 -> 750313975; device CM_passives:750313972 -> CM_passives:750313975
- U$1: value SSL.3IN_SILK -> STAR; device images:SSL.3IN_SILK -> images:STAR
- U$2: value STAR -> SSL.3IN_SILK; device images:STAR -> images:SSL.3IN_SILK
- U10: value MC74VHC1GT125 -> MC14504BDTG; device CM_IC:MC74VHC1GT125 -> MotorDriver:MC14504BDTG
- U11: value TCA9535_RTW_24 -> MAX31725MTA+; device MotorDriver:TCA9535_RTW_24 -> NR_IC:MAX31725MTA+
- U12: value MAX31725MTA+ -> TCA9535_RTW_24; device NR_IC:MAX31725MTA+ -> MotorDriver:TCA9535_RTW_24
- U15: value P82B715 -> MC74VHC1GT125; device CM_IC:P82B715 -> CM_IC:MC74VHC1GT125
- U16: value MC74VHC1GT125 -> PCA9515A; device CM_IC:MC74VHC1GT125 -> CM_IC:PCA9515A
- U9: value MC14504BDTG -> MC74VHC1GT125; device MotorDriver:MC14504BDTG -> CM_IC:MC74VHC1GT125
Connections:
- removed net N$17: Q6A.D, Q6B.G, R37.2
- removed net N$36: C40.1, C41.1, Q6B.D, U15.VCC
- net +3V3: now also C24.1, C34.1, C37.1, JP2.1, Q3P.S, R14.1, R23.2, R24.1, R28A.2, R28B.2, R28C.2, R28D.2, R3.2, U10.VCC, U11.VDD, U15.VIN, U16.VCC; no longer C25.1, C29.1, C35.1, JP1.1, Q5B.S, Q6B.S, R13.1, R15A.2, R15B.2, R15C.2, R15D.2, R2.2, R27.2, R28.1, R37.1, U12.VDD, U16.VIN, U9.VCC
- net +5V: now also C19.1, C28.1, C40.1, Q1P.S, Q2P.S, R12.1, R15.1, R16.1, R19.1, R25.2, R26.2, R27.2, R8.1, U10.VDD, U12.A0, U12.A1, U12.A2, U12.VCC, U9.VIN; no longer C17.1, C27.1, C38.1, Q1B.S, Q2B.S, R11.1, R14.1, R22.1, R23.1, R30.2, R32.2, R34.2, R7.1, U10.VIN, U11.A0, U11.A1, U11.A2, U11.VCC, U9.VDD
- net BIAS_GND: now also C17.1, R7.1, T1.7
- net BIAS_V: now also R7.2
- net DEBUG_5V: now also Q2P.D; no longer Q2B.D
- net DEC0: now also U12.P15; no longer U11.P15
- net DEC1: now also U12.P13; no longer U11.P13
- net DIR: now also U12.P12; no longer U11.P12
- net EXTERNAL_3V3: now also Q3P.D; no longer Q5B.D
- net EXTERNAL_KILL: now also Q2N.G, Q3N.G, R13.1, R22.1, U16.EN; no longer Q2A.G, Q5A.G, Q6A.G, R12.1, R26.1, R35.1
- net FB_5: now also R10.1, R8.2; no longer R7.2, R8.1
- net GND: now also C17.2, JP1.1, JP2.5, Q1N.S, Q2N.S, Q3N.S, R11.2, R13.2, R17.2, R20.1, R21.1, R22.2, R9.2, U10.MODE, U10.VSS, U11.A0, U11.A1, U11.A2, U11.EP, U12.EPAD, U15.OE, U9.GND, U9.OE; no longer C18.2, C41.2, JP1.5, JP2.1, Q1A.S, Q2A.S, Q5A.S, Q6A.S, R10.2, R12.2, R19.2, R24.1, R25.1, R26.2, R35.2, R8.2, U10.GND, U10.OE, U11.EPAD, U12.A0, U12.A1, U12.A2, U12.EP, U16.GND, U16.OE, U9.MODE, U9.VSS
- net I0: now also U12.P17; no longer U11.P17
- net I1: now also U12.P16; no longer U11.P16
- net IMUDR: now also U10.DIN; no longer U9.DIN
- net IMUINT1: now also U10.BIN; no longer U9.BIN
- net IMUINT2: now also U10.CIN; no longer U9.CIN
- net IMUINT3: now also U10.AIN; no longer U9.AIN
- net IMUINT4: now also U10.EIN; no longer U9.EIN
- net IMUINT5: now also U10.FIN; no longer U9.FIN
- net IOEINT: now also U15.Y; no longer U16.Y
- net M0: now also U12.P11; no longer U11.P11
- net M1: now also U12.P10; no longer U11.P10
- net N$10: now also C25.1, C26.1; no longer C19.1, C24.1
- net N$16: now also R29.1; no longer R34.1
- net N$18: now also Q3N.D, Q3P.G, R24.2; no longer Q5A.D, Q5B.G, R28.2
- net N$19: now also U10.AOUT, U12.P00; no longer U11.P00, U9.AOUT
- net N$20: now also R21.2; no longer R25.2
- net N$21: now also R20.2; no longer R24.2
- net N$22: now also U9.Y; no longer U10.Y
- net N$23: now also U10.BOUT, U12.P01; no longer U11.P01, U9.BOUT
- net N$25: now also U12.INT, U15.A; no longer U11.INT, U16.A
- net N$26: now also C38.1; no longer C37.1
- net N$28: now also U10.COUT, U12.P02; no longer U11.P02, U9.COUT
- net N$29: now also U10.DOUT, U12.P03; no longer U11.P03, U9.DOUT
- net N$30: now also U10.EOUT, U12.P04; no longer U11.P04, U9.EOUT
- net N$31: now also U10.FOUT, U12.P05; no longer U11.P05, U9.FOUT
- net N$32: now also R14.2; no longer R13.2
- net N$33: now also R27.1, U12.SDA; no longer R32.1, U11.SDA
- net N$34: now also R25.1, U12.SCL; no longer R29.1, U11.SCL
- net N$35: now also R26.1; no longer R30.1
- net N$37: now also Q1N.D, Q1P.G, R12.2; no longer Q1A.D, Q1B.G, R11.2
- net N$38: now also Q2N.D, Q2P.G, R15.2; no longer Q2A.D, Q2B.G, R14.2
- net N$48: now also C18.2, R10.2; no longer C17.2, R9.2
- net N$49: now also R2.2; no longer R3.2
- net N$5: now also C27.1; no longer C26.1
- net N$50: now also R2.1; no longer R3.1
- net N$52: now also T1.5
- net N$6: now also R23.1, U11.OS; no longer R27.1, U12.OS
- net N$7: now also JP1.2; no longer JP2.2
- net N$9: now also C29.1; no longer C28.1
- net NENBL: now also R19.2, U12.P07; no longer R23.2, U11.P07
- net NFAULT: now also R18.2, U12.P06; no longer R22.2, U11.P06
- net NSLEEP: now also U12.P14; no longer U11.P14
- net PI_5V: now also Q1P.D; no longer Q1B.D
- net PI_KILL: now also Q1N.G, R11.1; no longer Q1A.G, R10.1
- net RESET: now also JP2.2, R3.1; no longer JP1.2, R2.1
- net SCL: now also R28D.1, U11.SCL; no longer R15D.1, U12.SCL, U15.SX
- net SCL_BUFF: now also R28B.1; no longer R15B.1, U15.LX
- net SDA: now also R28C.1, U11.SDA; no longer R15C.1, U12.SDA, U15.SY
- net SDA_BUFF: now also R28A.1; no longer R15A.1, U15.LY
- net STEPFREQ: now also U9.A; no longer U10.A
- net SWDCLK: now also JP2.4; no longer JP1.4
- net SWDIO: now also JP2.6; no longer JP1.6
- net VREFA: now also C35.1; no longer C34.1
- net V_SENSE: now also R16.2, R17.1; no longer R18.2, R19.1
Other:
- moved on the sheet: C1, C16, C17, C18, C19, C20, C21, C22, C23, C24, C25, C26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
