File: CAD/eagle/STARduino/starduino.brd (EAGLE design)
At the start: 101.6 x 38.1 mm, 123 parts, among them J1 J30J-9J30, J2 MICRO_SD, J3 J30J-15J30, J4 J30J-31J30, J5 RPI-ZERO, J6 RPI-CSI, Q1 FDG8842CZ, Q2 FDG8842CZ, Q3 DMMT5401, Q4 DMG2305UX, Q5 FDG8842CZ, Q6 FDG8842CZ, T1 750313972, U1 LT8301, U10 MC74VHC1GT125DT, U11 TCA9535_RTW_24, U12 MAX31725MTA+, U13 BMX055, U14 DRV8846RGER, U15 P82B715, U16 MC74VHC1GT125DT, U17 PCA9306DCT, U2 LT3465/A, U3 LTC3112FE, U4 DS3231MZ+, U5 MT25QL01GBBB8ESF-0AAT, U6 ATSAMD21G18, U7 MIC5216, U8 ADXL375BCCZ, U9 MC14504BDTG

Commit message: Fixed STEPFREQ schematic bug.
Connections:
- net STEPFREQ: now also U6.13; no longer U6.7
Changed lines of the file:
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@@
 <?xml version="1.0" encoding="utf-8"?>
 <!DOCTYPE eagle SYSTEM "eagle.dtd">
-<eagle version="6.5.0">
+<eagle version="7.7.0">
 <drawing>
 <settings>
@@
 <layer number="59" name="tCarbon" color="7" fill="1" visible="no" active="no"/>
 <layer number="60" name="bCarbon" color="7" fill="1" visible="no" active="no"/>
-<layer number="90" name="Modules" color="5" fill="1" visible="no" active="yes"/>
+<layer number="90" name="Modules" color="5" fill="1" visible="no" active="no"/>
 <layer number="91" name="Nets" color="2" fill="1" visible="no" active="no"/>
 <layer number="92" name="Busses" color="1" fill="1" visible="no" active="no"/>
@@
 <pass name="Default">
 <param name="RoutingGrid" value="50mil"/>
+<param name="AutoGrid" value="1"/>
+<param name="Efforts" value="0"/>
+<param name="TopRouterVariant" value="1"/>
 <param name="tpViaShape" value="round"/>
 <param name="PrefDir.1" value="|"/>
@@
 <contactref element="U10" pad="1"/>
 <contactref element="U10" pad="3"/>
-<contactref element="U10" pad="3"/>
-<contactref element="U16" pad="3"/>
 <contactref element="U16" pad="3"/>
 <contactref element="U16" pad="1"/>
@@
 <signal name="STEPFREQ">
 <contactref element="U10" pad="2"/>
-<contactref element="U6" pad="7"/>
-<wire x1="-42.3418" y1="16.256" x2="114.3" y2="21.52" width="0" layer="19" extent="1-1"/>
+<contactref element="U6" pad="13"/>
+<wire x1="-40.8432" y1="12.2682" x2="114.3" y2="21.52" width="0" layer="19" extent="1-1"/>
 </signal>
 <signal name="NENBL">
