File: CAD/eagle/STARduino/starduino.brd (EAGLE design)
At the start: 101.6 x 38.1 mm, 123 parts, among them J1 J30J-9J30, J2 MICRO_SD, J3 J30J-15J30, J4 J30J-31J30, J5 RPI-ZERO, J6 RPI-CSI, Q1 FDG8842CZ, Q2 FDG8842CZ, Q3 DMMT5401, Q4 DMG2305UX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

Commit message: Board routing
Parts:
- moved U9 73.5 mm to (114.3, 15.2)
- moved U17 65.2 mm to (108.8, 22.1), turned to 270 degrees
- moved R29 63.2 mm to (123.2, 16.5)
- moved R30 63.2 mm to (128.3, 19.1)
- moved R32 63.2 mm to (128.3, 16.5)
- moved U16 63.2 mm to (128.3, 22.9)
- moved U11 58.0 mm to (114.3, 22.9), turned to 90 degrees
- moved R23 16.3 mm to (109.8, 30.0), turned to 180 degrees
- moved R22 14.8 mm to (109.8, 28.6), turned to 180 degrees
- moved C39 13.7 mm to (110.3, 31.4), turned to 180 degrees
- moved C37 12.2 mm to (109.8, 27.2), turned to 180 degrees
- moved U14 9.49 mm to (114.3, 28.3), turned to 180 degrees
- moved C38 8.61 mm to (109.8, 24.5)
- moved R34 7.81 mm to (109.8, 25.9), turned to 180 degrees
- moved U10 7.01 mm to (121.0, 22.2), turned to 270 degrees
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Connections:
- net DEC0: now also U11.15; no longer U11.10
- net DEC1: now also U11.13; no longer U11.11
- net I0: now also U11.17; no longer U11.16
- net I1: now also U11.16; no longer U11.17
- net M0: now also U11.7; no longer U11.14
- net M1: now also U11.10; no longer U11.15
- net NFAULT: now also U11.11; no longer U11.13
- net NSLEEP: now also U11.14; no longer U11.7
Routing:
- net MA2: track 0.00 -> 23.9 mm
- net MA1: track 0.00 -> 23.9 mm
- net NENBL: track 0.00 -> 20.0 mm, vias 0 -> 3
- net MB2: track 0.00 -> 18.8 mm
- net MB1: track 0.00 -> 18.2 mm
- net +5V: track 1.66 -> 18.8 mm, vias 0 -> 2
- net PRESSURE_IN: track 0.00 -> 11.6 mm
- net SCL_BUFF: track 0.00 -> 10.4 mm
- net NFAULT: track 0.00 -> 9.30 mm, vias 0 -> 2
- net N$26: track 0.00 -> 9.22 mm, vias 0 -> 2
- net SDA_BUFF: track 0.00 -> 6.69 mm
- net N$34: track 0.00 -> 6.64 mm
- net EXTERNAL_3V3: track 0.00 -> 5.76 mm
- net GND: track 15.5 -> 20.1 mm
- net DIR: track 0.00 -> 3.44 mm, vias 0 -> 1
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
Commit message: Fixed Arduino fuckery
Connections:
- net MISO: now also U6.21; no longer U6.8
- net SYNC: now also U6.24; no longer U6.21
Changed lines of the file:
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@@
 <?xml version="1.0" encoding="utf-8"?>
 <!DOCTYPE eagle SYSTEM "eagle.dtd">
-<eagle version="6.5.0">
+<eagle version="7.7.0">
 <drawing>
 <settings>
@@
 <pass name="Default">
 <param name="RoutingGrid" value="50mil"/>
+<param name="AutoGrid" value="1"/>
+<param name="Efforts" value="0"/>
+<param name="TopRouterVariant" value="1"/>
 <param name="tpViaShape" value="round"/>
 <param name="PrefDir.1" value="|"/>
@@
 <contactref element="J2" pad="7"/>
 <contactref element="U5" pad="8"/>
-<contactref element="U6" pad="8"/>
-<wire x1="-42.3418" y1="15.748" x2="55.64" y2="7.21" width="0" layer="19" extent="1-1"/>
-<wire x1="-33.655" y1="58.9" x2="-42.3418" y2="15.748" width="0" layer="19" extent="1-1"/>
+<contactref element="U6" pad="21"/>
+<wire x1="-36.8554" y1="12.2682" x2="55.64" y2="7.21" width="0" layer="19" extent="1-1"/>
+<wire x1="-33.655" y1="58.9" x2="-36.8554" y2="12.2682" width="0" layer="19" extent="1-1"/>
 </signal>
 <signal name="TX1">
@@
 </signal>
 <signal name="SYNC">
-<contactref element="U6" pad="21"/>
 <contactref element="J5" pad="37"/>
-<wire x1="-36.8554" y1="12.2682" x2="78.74" y2="33.147" width="0" layer="19" extent="1-1"/>
+<contactref element="U6" pad="24"/>
+<wire x1="-35.3568" y1="12.2682" x2="78.74" y2="33.147" width="0" layer="19" extent="1-1"/>
 </signal>
 <signal name="EXTERNAL_KILL">

Commit message: layout stuff
Parts:
- moved U13 148.8 mm to (70.8, 16.3), turned to 90 degrees
- moved C35 147.0 mm to (67.9, 20.2), turned to 180 degrees
- moved C33 146.3 mm to (67.9, 18.9), turned to 180 degrees
- moved C36 99.2 mm to (71.1, -2.54)
- moved R27 99.2 mm to (67.3, -2.54)
- moved U12 98.9 mm to (69.0, -5.95)
- moved R26 89.5 mm to (90.0, 35.4), turned to 270 degrees
- moved Q5 87.8 mm to (92.2, 35.6)
- moved R28 86.1 mm to (94.3, 35.6), turned to 90 degrees
- moved JP2 66.7 mm to (31.6, 3.57)
- moved R32 57.5 mm to (71.4, 24.9), turned to 180 degrees
- moved U16 56.9 mm to (71.4, 21.2), turned to 90 degrees
- moved R30 56.8 mm to (71.4, 18.9), turned to 180 degrees
- moved R29 52.2 mm to (71.4, 23.5), turned to 180 degrees
- moved U10 48.1 mm to (73.3, 27.8), turned to 90 degrees
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Connections:
- net IMUDR: now also U9.9; no longer U9.3
- net IMUINT3: now also U9.3; no longer U9.9
Routing:
- net SDA_BUFF: track 6.69 -> 51.4 mm, vias 0 -> 1
- net SCL_BUFF: track 10.4 -> 51.6 mm, vias 0 -> 1
- net MA1: track 23.9 -> 49.5 mm, vias 0 -> 2
- net +3V3: track 0.00 -> 17.8 mm
- net PRESSURE_IN: track 11.6 -> 29.0 mm, vias 0 -> 2
- net IMUINT2: track 0.00 -> 15.5 mm, vias 0 -> 2
- net M0: track 0.00 -> 15.2 mm, vias 0 -> 2
- net M1: track 0.00 -> 14.7 mm, vias 0 -> 2
- net N$31: track 0.00 -> 14.2 mm, vias 0 -> 2
- net +5V: track 18.8 -> 32.7 mm
- net MA2: track 23.9 -> 37.4 mm, vias 0 -> 2
- net N$30: track 0.00 -> 12.5 mm, vias 0 -> 2
- net MB1: track 18.2 -> 29.9 mm
- net DIR: track 3.44 -> 14.1 mm, vias 1 -> 2
- net IMUINT1: track 0.00 -> 10.5 mm, vias 0 -> 1
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
Commit message: routing
Parts:
- moved C31 156.0 mm to (74.4, 10.7), turned to 180 degrees
- moved C32 152.1 mm to (74.4, 12.1), turned to 180 degrees
- moved C30 149.0 mm to (70.6, 6.67)
- moved U8 148.2 mm to (70.6, 10.4), turned to 180 degrees
- moved C27 95.9 mm to (30.6, 30.2)
- moved U7 94.5 mm to (30.7, 27.9), turned to 90 degrees
- moved C29 92.2 mm to (31.1, 25.3), turned to 180 degrees
- moved R18 73.8 mm to (64.8, 48.3)
- moved R19 73.8 mm to (64.8, 50.8)
- moved R20 73.8 mm to (76.2, 47.0)
- moved R21 73.8 mm to (76.2, 49.5)
- moved C15 35.2 mm to (36.8, 22.8)
- moved C3 35.2 mm to (42.9, 26.7)
- moved L1 35.2 mm to (39.1, 27.5)
- moved R4 35.2 mm to (41.4, 23.7)
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Routing:
- net +3V3: track 17.8 -> 28.1 mm, vias 0 -> 2
- net IMUINT3: track 6.01 -> 14.7 mm, vias 1 -> 2
- net LED_V: track 37.7 -> 29.7 mm
- net IMUINT4: track 0.00 -> 7.43 mm, vias 0 -> 2
- net IMUINT1: track 10.5 -> 17.9 mm, vias 1 -> 2
- net IMUDR: track 0.00 -> 5.91 mm
- net LED_GND: track 34.5 -> 29.7 mm
- net GND: track 24.8 -> 27.1 mm, vias 4 -> 5
- net SCL: track 0.00 -> 1.24 mm, vias 0 -> 1

Commit message: stuff
Parts:
- removed C28: 1μF, resistor:C0603
- removed F1: 1206L150THWR, adafruit:R1206
- removed Q3: DMMT5401, transistor-pnp:SOT-26
- removed Q4: DMG2305UX, microbuilder:SOT23-R
- removed R15: 10k, resistor:R0603
- removed R16: 47k, resistor:R0603
- moved R13 95.9 mm to (34.5, 11.2), turned to 180 degrees
- moved C25 94.1 mm to (34.5, 9.60), turned to 180 degrees
- moved U6 91.9 mm to (53.3, 25.4)
- moved U5 88.8 mm to (37.9, 17.6), turned to 270 degrees
- moved XTAL1 83.9 mm to (22.9, 63.5)
- moved C10 83.5 mm to (21.6, 76.2)
- moved C19 83.5 mm to (31.8, 73.7)
- moved C20 83.5 mm to (31.8, 69.8)
- moved C21 83.5 mm to (36.8, 69.8)
- moved C22 83.5 mm to (36.8, 73.7)
- moved C23 83.5 mm to (26.7, 73.7)
- moved C24 83.5 mm to (25.4, 71.1)
- moved C26 83.5 mm to (40.6, 64.8)
- moved C34 83.5 mm to (41.9, 73.7)
- moved C7 83.5 mm to (21.6, 61.0)
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Connections:
- removed net N$53: J5.2, J5.4, Q3.5, Q4.3
- removed net N$54: Q3.4, Q4.1, R16.1
- removed net N$55: Q3.1, Q3.2, Q3.3, R15.1
- removed net N$56: C28.1, F1.2, Q3.6, Q4.2
- net +5V: no longer F1.1
- net GND: no longer C28.2, R15.2, R16.2
- net PI_5V: now also J5.2, J5.4
Routing:
- net +3V3: track 28.1 -> 86.9 mm, vias 2 -> 4
- net +5V: track 32.7 -> 76.5 mm
- net SCL: track 1.24 -> 40.8 mm, vias 1 -> 2
- net SDA: track 1.51 -> 27.2 mm, vias 1 -> 2
- net PRESSURE_IN: track 29.0 -> 49.7 mm
- net EXTERNAL_KILL: track 3.14 -> 17.0 mm
- net STEPFREQ: track 0.00 -> 10.8 mm, vias 0 -> 1
- net EXTERNAL_3V3: track 7.76 -> 11.8 mm
- net PB03: track 0.00 -> 3.10 mm, vias 0 -> 1
- net PB02: track 0.00 -> 2.80 mm, vias 0 -> 1
- net IMUINT4: track 7.43 -> 8.89 mm
- net LED_V: track 29.7 -> 28.5 mm, vias 1 -> 0
- net FB_5: track 13.7 -> 14.8 mm
- net LED_GND: track 29.7 -> 28.7 mm, vias 1 -> 0
- net SCL_BUFF: track 51.6 -> 51.0 mm
- removed copper zone on layer 1, net LED_GND
- removed copper zone on layer 1, net LED_V

Commit message: Package stuff
Parts:
- moved C7 56.7 mm to (62.1, 21.3)
- moved XTAL1 55.3 mm to (59.5, 22.0), turned to 270 degrees
- moved C8 53.9 mm to (62.1, 22.8)
- moved R4 17.3 mm to (34.9, 13.8), turned to 180 degrees
- moved C3 17.2 mm to (41.5, 14.5), turned to 270 degrees
- moved U2 13.6 mm to (34.3, 16.1), turned to 270 degrees
- moved L1 11.1 mm to (38.7, 16.7), turned to 90 degrees
- moved C15 10.0 mm to (34.0, 18.5), turned to 0 degrees
- moved U5 8.09 mm to (39.5, 25.6)
- moved J2 0.79 mm to (60.3, 9.37)
- moved Q6 0.40 mm to (64.9, 24.2)
- moved C40 0.32 mm to (62.6, 28.7)
- moved R37 0.32 mm to (62.6, 25.5)
- moved C41 0.24 mm to (61.1, 28.7)
- moved R35 0.24 mm to (61.1, 25.5)
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Connections:
- removed net USB_D+: U6.34
- removed net USB_D-: U6.33
- net USB_D_N: now also U6.33
- net USB_D_P: now also U6.34
Routing:
- net EXTERNAL_KILL: track 17.0 -> 11.5 mm
- net +3V3: track 86.9 -> 92.1 mm

Commit message: layout stuff
Parts:
- TP1, TP2: value TESTPOINT -> TESTPOINT1.5MM; device CM_passives:TP-2MM -> CM_passives:TP-1.5MM
- U10, U16: value MC74VHC1GT125DT -> MC74VHC1GT125; device MotorDriver:TSOP-5 -> CM_IC:SC-70-5
- moved R10 55.4 mm to (28.3, 22.2), turned to 90 degrees
- moved R11 54.9 mm to (32.5, 22.2), turned to 90 degrees
- moved R21 45.9 mm to (47.0, 14.1), turned to 180 degrees
- moved R20 45.0 mm to (47.0, 12.7), turned to 180 degrees
- moved L5 42.2 mm to (48.9, 20.8), turned to 90 degrees
- moved L3 40.0 mm to (53.3, 18.8)
- moved L4 36.9 mm to (58.0, 29.9), turned to 180 degrees
- moved C10 24.3 mm to (24.1, 52.1)
- moved R1 23.2 mm to (24.1, 47.0)
- moved R2 23.0 mm to (24.1, 49.5)
- moved R13 18.4 mm to (33.6, 29.5), turned to 270 degrees
- moved C25 10.3 mm to (34.0, 19.9)
- moved TP1 5.92 mm to (22.9, 17.3)
- moved TP2 5.36 mm to (21.0, 17.3)
- moved C16 1.27 mm to (10.8, 15.8)
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Connections:
- net PI_D_N: now also J3.7; no longer J3.8
- net PI_D_P: now also J3.8; no longer J3.7
Routing:
- net USB_D_P: track 0.00 -> 45.6 mm, vias 0 -> 2
- net USB_D_N: track 0.00 -> 44.7 mm, vias 0 -> 2
- net PI_D_N: track 0.00 -> 24.9 mm, vias 0 -> 1
- net PI_D_P: track 0.00 -> 24.8 mm, vias 0 -> 1
- net XIN32: track 0.00 -> 5.49 mm
- net XOUT32: track 0.00 -> 4.59 mm
- net +5V: track 76.5 -> 79.2 mm
- net +3V3: track 92.1 -> 93.9 mm
- net N$22: track 12.2 -> 13.9 mm

Commit message: layout progress
Parts:
- moved C23 61.8 mm to (47.2, 15.4), turned to 270 degrees
- moved C19 59.9 mm to (45.8, 15.4), turned to 270 degrees
- moved C34 58.7 mm to (61.7, 18.4)
- moved FB1 57.4 mm to (57.7, 20.7), turned to 270 degrees
- moved C24 57.0 mm to (47.2, 18.5), turned to 90 degrees
- moved C22 55.7 mm to (44.4, 18.5), turned to 90 degrees
- moved C21 55.0 mm to (44.4, 15.4), turned to 270 degrees
- moved L6 54.4 mm to (58.5, 18.4)
- moved C20 53.2 mm to (45.8, 18.5), turned to 90 degrees
- moved C26 48.1 mm to (52.1, 18.0), turned to 180 degrees
- moved C10 41.0 mm to (34.3, 12.3), turned to 180 degrees
- moved R2 40.0 mm to (34.3, 10.8), turned to 180 degrees
- moved R1 39.0 mm to (34.3, 9.29)
- moved R19 32.4 mm to (64.8, 18.4), turned to 180 degrees
- moved R18 27.5 mm to (65.3, 20.8), turned to 270 degrees
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Connections:
- removed net PRESSURE_IN: J4.11, U6.11
Routing:
- net SCL: track 41.0 -> 117.7 mm, vias 2 -> 8
- net SDA: track 27.2 -> 89.8 mm, vias 2 -> 6
- net EXTERNAL_KILL: track 11.5 -> 70.9 mm
- net LED_V: track 28.5 -> 83.4 mm, vias 0 -> 1
- net PRESSURE_IN: track 49.7 -> 0.00 mm, vias 2 -> 0
- net LED_GND: track 28.7 -> 73.9 mm
- net +5V: track 79.2 -> 122.9 mm, vias 2 -> 7
- net MISO: track 0.00 -> 41.3 mm, vias 0 -> 3
- net MOSI: track 0.00 -> 39.6 mm, vias 0 -> 2
- net SCK: track 0.00 -> 35.4 mm, vias 0 -> 2
- net LED_CTRL: track 0.00 -> 34.7 mm, vias 0 -> 2
- net +3V3: track 93.9 -> 121.6 mm, vias 4 -> 7
- net PA27: track 0.00 -> 26.4 mm, vias 0 -> 2
- net RESET: track 0.00 -> 24.9 mm, vias 0 -> 2
- net PB22: track 0.00 -> 21.7 mm, vias 0 -> 2
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- added copper zone on layer 1, net +3V3
