File: CAD/eagle/Debug_Breakout/Debug_Breakout.sch (EAGLE design)
At the start: 16 parts, among them Q1 CM1213A-02SR, Q2 CM1213A-02SR

Commit message: Finished STAR debug board.
Parts:
- added U$1: SSL.3IN_SILK, images:SSL.3IN_SILK
- added U$2: STAR, images:STAR
Connections:
- removed net N$1: MCU.D+, Q1.CH2, R1B.2
- removed net N$2: MCU.D-, Q1.CH1, R1C.2
- removed net N$3: PI.D+, Q2.CH2, R2B.2
- removed net N$4: PI.D-, Q2.CH1, R2C.2
- removed net N$6: PI.GND, Q2.GND
- removed net N$7: MCU.GND, Q1.GND
- new net MCU_D_N: MCU.D-, Q1.CH2, R1C.2
- new net MCU_D_P: MCU.D+, Q1.CH1, R1B.2
- new net PICONN_D_N: PI.D-, Q2.CH2, R2C.2
- new net PICONN_D_P: PI.D+, Q2.CH1, R2B.2
- net GND: now also MCU.GND, PI.GND, Q1.GND, Q2.GND
Changed lines of the file:
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@@
 <layer number="97" name="Info" color="7" fill="1" visible="yes" active="yes"/>
 <layer number="98" name="Guide" color="6" fill="1" visible="yes" active="yes"/>
+<layer number="99" name="SpiceOrder" color="5" fill="1" visible="yes" active="yes"/>
 <layer number="100" name="Muster" color="7" fill="1" visible="no" active="no"/>
 <layer number="101" name="Patch_Top" color="12" fill="4" visible="yes" active="yes"/>
@@
 <part name="GND5" library="supply1" deviceset="GND" device=""/>
 <part name="GND6" library="supply1" deviceset="GND" device=""/>
+<part name="GND7" library="supply1" deviceset="GND" device=""/>
+<part name="GND8" library="supply1" deviceset="GND" device=""/>
+<part name="U$1" library="images" deviceset="SSL" device=".3IN_SILK" value="SSL.3IN_SILK"/>
+<part name="U$2" library="images" deviceset="STAR" device=""/>
 </parts>
 <sheets>
@@
 <instance part="GND5" gate="1" x="137.16" y="114.3"/>
 <instance part="GND6" gate="1" x="180.34" y="190.5"/>
+<instance part="GND7" gate="1" x="76.2" y="152.4"/>
+<instance part="GND8" gate="1" x="76.2" y="91.44"/>
+<instance part="U$1" gate="G$1" x="269.24" y="45.72"/>
+<instance part="U$2" gate="G$1" x="254" y="38.1"/>
 </instances>
 <busses>
 </busses>
 <nets>
-<net name="N$1" class="0">
-<segment>
+<net name="MCU_D_P" class="0">
+<segment>
+<pinref part="MCU" gate="G$1" pin="D+"/>
+<wire x1="73.66" y1="180.34" x2="53.34" y2="180.34" width="0.1524" layer="91"/>
+<wire x1="53.34" y1="180.34" x2="53.34" y2="172.72" width="0.1524" layer="91"/>
+<pinref part="R1" gate="B" pin="2"/>
+<wire x1="53.34" y1="172.72" x2="48.26" y2="172.72" width="0.1524" layer="91"/>
+<pinref part="Q1" gate="G$1" pin="CH1"/>
+<wire x1="48.26" y1="172.72" x2="45.72" y2="172.72" width="0.1524" layer="91"/>
+<wire x1="50.8" y1="162.56" x2="48.26" y2="162.56" width="0.1524" layer="91"/>
+<wire x1="48.26" y1="162.56" x2="48.26" y2="172.72" width="0.1524" layer="91"/>
+<junction x="48.26" y="172.72"/>
+</segment>
+</net>
+<net name="MCU_D_N" class="0">
+<segment>
+<pinref part="MCU" gate="G$1" pin="D-"/>
+<wire x1="45.72" y1="182.88" x2="68.58" y2="182.88" width="0.1524" layer="91"/>
+<pinref part="R1" gate="C" pin="2"/>
 <pinref part="Q1" gate="G$1" pin="CH2"/>
+<wire x1="68.58" y1="182.88" x2="73.66" y2="182.88" width="0.1524" layer="91"/>
 <wire x1="66.04" y1="162.56" x2="68.58" y2="162.56" width="0.1524" layer="91"/>
-<wire x1="68.58" y1="162.56" x2="68.58" y2="180.34" width="0.1524" layer="91"/>
-<pinref part="MCU" gate="G$1" pin="D+"/>
-<wire x1="68.58" y1="180.34" x2="73.66" y2="180.34" width="0.1524" layer="91"/>
-<wire x1="68.58" y1="180.34" x2="53.34" y2="180.34" width="0.1524" layer="91"/>
-<wire x1="53.34" y1="180.34" x2="53.34" y2="172.72" width="0.1524" layer="91"/>
-<junction x="68.58" y="180.34"/>
-<pinref part="R1" gate="B" pin="2"/>
-<wire x1="53.34" y1="172.72" x2="45.72" y2="172.72" width="0.1524" layer="91"/>
-</segment>
-</net>
-<net name="N$2" class="0">
-<segment>
-<pinref part="Q1" gate="G$1" pin="CH1"/>
-<wire x1="50.8" y1="162.56" x2="48.26" y2="162.56" width="0.1524" layer="91"/>
-<wire x1="48.26" y1="162.56" x2="48.26" y2="182.88" width="0.1524" layer="91"/>
-<pinref part="MCU" gate="G$1" pin="D-"/>
-<wire x1="48.26" y1="182.88" x2="73.66" y2="182.88" width="0.1524" layer="91"/>
-<pinref part="R1" gate="C" pin="2"/>
-<wire x1="48.26" y1="182.88" x2="45.72" y2="182.88" width="0.1524" layer="91"/>
-<junction x="48.26" y="182.88"/>
+<wire x1="68.58" y1="162.56" x2="68.58" y2="182.88" width="0.1524" layer="91"/>
+<junction x="68.58" y="182.88"/>
 </segment>
 </net>
@@
 <wire x1="180.34" y1="193.04" x2="193.04" y2="193.04" width="0.1524" layer="91"/>
 </segment>
+<segment>
+<pinref part="Q1" gate="G$1" pin="GND"/>
+<wire x1="58.42" y1="154.94" x2="71.12" y2="154.94" width="0.1524" layer="91"/>
+<wire x1="71.12" y1="154.94" x2="71.12" y2="175.26" width="0.1524" layer="91"/>
+<pinref part="MCU" gate="G$1" pin="GND"/>
+<wire x1="71.12" y1="175.26" x2="73.66" y2="175.26" width="0.1524" layer="91"/>
+<pinref part="GND7" gate="1" pin="GND"/>
+<wire x1="71.12" y1="154.94" x2="76.2" y2="154.94" width="0.1524" layer="91"/>
+<junction x="71.12" y="154.94"/>
+</segment>
+<segment>
+<pinref part="Q2" gate="G$1" pin="GND"/>
+<wire x1="58.42" y1="93.98" x2="71.12" y2="93.98" width="0.1524" layer="91"/>
+<wire x1="71.12" y1="93.98" x2="71.12" y2="114.3" width="0.1524" layer="91"/>
+<pinref part="PI" gate="G$1" pin="GND"/>
+<wire x1="71.12" y1="114.3" x2="73.66" y2="114.3" width="0.1524" layer="91"/>
+<pinref part="GND8" gate="1" pin="GND"/>
+<wire x1="71.12" y1="93.98" x2="76.2" y2="93.98" width="0.1524" layer="91"/>
+<junction x="71.12" y="93.98"/>
+</segment>
 </net>
 <net name="PI_D_N" class="0">
@@
 </segment>
 </net>
-<net name="N$3" class="0">
-<segment>
+<net name="PICONN_D_P" class="0">
+<segment>
+<pinref part="PI" gate="G$1" pin="D+"/>
+<wire x1="73.66" y1="119.38" x2="53.34" y2="119.38" width="0.1524" layer="91"/>
+<wire x1="53.34" y1="119.38" x2="53.34" y2="111.76" width="0.1524" layer="91"/>
+<pinref part="R2" gate="B" pin="2"/>
+<wire x1="53.34" y1="111.76" x2="48.26" y2="111.76" width="0.1524" layer="91"/>
+<pinref part="Q2" gate="G$1" pin="CH1"/>
+<wire x1="48.26" y1="111.76" x2="45.72" y2="111.76" width="0.1524" layer="91"/>
+<wire x1="50.8" y1="101.6" x2="48.26" y2="101.6" width="0.1524" layer="91"/>
+<wire x1="48.26" y1="101.6" x2="48.26" y2="111.76" width="0.1524" layer="91"/>
+<junction x="48.26" y="111.76"/>
+</segment>
+</net>
+<net name="PICONN_D_N" class="0">
+<segment>
+<pinref part="PI" gate="G$1" pin="D-"/>
+<pinref part="R2" gate="C" pin="2"/>
+<wire x1="73.66" y1="121.92" x2="68.58" y2="121.92" width="0.1524" layer="91"/>
 <pinref part="Q2" gate="G$1" pin="CH2"/>
+<wire x1="68.58" y1="121.92" x2="45.72" y2="121.92" width="0.1524" layer="91"/>
 <wire x1="66.04" y1="101.6" x2="68.58" y2="101.6" width="0.1524" layer="91"/>
-<wire x1="68.58" y1="101.6" x2="68.58" y2="119.38" width="0.1524" layer="91"/>
-<pinref part="PI" gate="G$1" pin="D+"/>
-<wire x1="73.66" y1="119.38" x2="68.58" y2="119.38" width="0.1524" layer="91"/>
-<wire x1="68.58" y1="119.38" x2="53.34" y2="119.38" width="0.1524" layer="91"/>
-<wire x1="53.34" y1="119.38" x2="53.34" y2="111.76" width="0.1524" layer="91"/>
-<junction x="68.58" y="119.38"/>
-<pinref part="R2" gate="B" pin="2"/>
-<wire x1="53.34" y1="111.76" x2="45.72" y2="111.76" width="0.1524" layer="91"/>
-</segment>
-</net>
-<net name="N$4" class="0">
-<segment>
-<pinref part="PI" gate="G$1" pin="D-"/>
-<wire x1="73.66" y1="121.92" x2="48.26" y2="121.92" width="0.1524" layer="91"/>
-<pinref part="Q2" gate="G$1" pin="CH1"/>
-<wire x1="50.8" y1="101.6" x2="48.26" y2="101.6" width="0.1524" layer="91"/>
-<wire x1="48.26" y1="101.6" x2="48.26" y2="121.92" width="0.1524" layer="91"/>
-<pinref part="R2" gate="C" pin="2"/>
-<wire x1="48.26" y1="121.92" x2="45.72" y2="121.92" width="0.1524" layer="91"/>
-<junction x="48.26" y="121.92"/>
+<wire x1="68.58" y1="101.6" x2="68.58" y2="121.92" width="0.1524" layer="91"/>
+<junction x="68.58" y="121.92"/>
 </segment>
 </net>
@@
 </segment>
 </net>
-<net name="N$6" class="0">
-<segment>
-<pinref part="Q2" gate="G$1" pin="GND"/>
-<wire x1="58.42" y1="93.98" x2="58.42" y2="91.44" width="0.1524" layer="91"/>
-<wire x1="58.42" y1="91.44" x2="71.12" y2="91.44" width="0.1524" layer="91"/>
-<wire x1="71.12" y1="91.44" x2="71.12" y2="114.3" width="0.1524" layer="91"/>
-<pinref part="PI" gate="G$1" pin="GND"/>
-<wire x1="71.12" y1="114.3" x2="73.66" y2="114.3" width="0.1524" layer="91"/>
-</segment>
-</net>
-<net name="N$7" class="0">
-<segment>
-<pinref part="Q1" gate="G$1" pin="GND"/>
-<wire x1="58.42" y1="154.94" x2="58.42" y2="152.4" width="0.1524" layer="91"/>
-<wire x1="58.42" y1="152.4" x2="71.12" y2="152.4" width="0.1524" layer="91"/>
-<wire x1="71.12" y1="152.4" x2="71.12" y2="175.26" width="0.1524" layer="91"/>
-<pinref part="MCU" gate="G$1" pin="GND"/>
-<wire x1="71.12" y1="175.26" x2="73.66" y2="175.26" width="0.1524" layer="91"/>
-</segment>
-</net>
